File: Main_Board/_autosave-Main_Board.sch (KiCad schematic (older format))
At the start: 58 parts, among them IC1 AZ1085CD-3.3TRG1, U1 STM32L152ZCTx, U2 LM386

Commit message: Revert first symbol rescue change.
This reverts commit da5e3b956d62bf000f607909d73018914190f8b5.
Parts:
- removed C17, C20: 22u, symbol Device:C_Small
- removed C18, C19: 100n, SamacSys_Parts:CAPC2012X95N, symbol Device:C_Small
- removed C21: C_Small, symbol Device:C_Small
- removed C22: 10u, symbol Device:C
- removed C23: 22u, symbol Device:C
- removed HallSensorHeader1: Conn_01x04_Male, Connector_PinHeader_2.54mm:PinHeader_1x04_P2.54mm_Vertical, symbol Connector:Conn_01x04_Male
- removed IC1: AZ1085CD-3.3TRG1, AZ1085CD33TRG1, symbol SamacSys_Parts:AZ1085CD-3.3TRG1
- removed LED_Header1, LED_Header2: Conn_01x09_Male, Connector_PinHeader_2.54mm:PinHeader_1x09_P2.54mm_Vertical, symbol Connector:Conn_01x09_Male
- removed SD_CARD1: 47352-1001, 47352-1001, symbol SamacSys_Parts:47352-1001
- removed UARTHeader1: Conn_01x02_Male, Connector_PinHeader_2.54mm:PinHeader_1x02_P2.54mm_Vertical, symbol Connector:Conn_01x02_Male
- added 5V-3V3: ZLDO1117K33TC, TO-252_1, symbol SamacSys_Parts:ZLDO1117K33TC
- added C11: 100n, SamacSys_Parts:CAPC1005X55N, symbol Device:C
- added Crst0: C, Capacitor_SMD:C_1812_4532Metric_Pad1.57x3.40mm_HandSolder, symbol Device:C
- added HALLOUT1, HALLSEL[0]1, HALLSEL[1]1, HALLSEL[2]1, UART_Rx1, UART_Tx1: MountingHole_Pad, MountingHole:MountingHole_2.7mm_Pad, symbol Mechanical:MountingHole_Pad
- added R1: R_Small, Resistor_THT:R_Axial_DIN0309_L9.0mm_D3.2mm_P12.70mm_Horizontal, symbol Device:R_Small
- added SEG0_7SEG1, SEG0_LED1, SEG1_7SEG1, SEG1_LED1, SEG2_7SEG1, SEG2_LED1, SEG3_7SEG1, SEG3_LED1, SEG4_7SEG1, SEG4_LED1, SEG5_7SEG1, SEG5_LED1, SEG6_7SEG1, SEG6_LED1, SEG7_7SEG1, SEG7_LED1, SEG8_7SEG1, SEG8_LED1: MountingHole_Pad, MountingHole:MountingHole_2.5mm_Pad, symbol Mechanical:MountingHole_Pad
- added nRST1: SW_MEC_5G, Button_Switch_SMD:Panasonic_EVQPUL_EVQPUC, symbol Switch:SW_MEC_5G
- C0, C1, C10, C2, C3, C4, C5, C6, C7, C8, C9: footprint SamacSys_Parts:CAPC2012X95N -> SamacSys_Parts:CAPC1005X55N
- C12, C14, C15: footprint SamacSys_Parts:CAPC2012X95N -> (none)
- C13: footprint SamacSys_Parts:CAPC2012X140N -> (none)
- C16: footprint Capacitor_THT:CP_Radial_D4.0mm_P2.00mm -> (none)
- CA1: footprint SamacSys_Parts:CAPC2012X140N -> SamacSys_Parts:CAPC1005X55N
- CSET7SEG1, CSETLED1: value 47p -> C_Small; footprint SamacSys_Parts:CAPC2012X75N -> Capacitor_SMD:C_1812_4532Metric_Pad1.57x3.40mm_HandSolder
- R4, R5, R6: footprint Resistor_THT:R_Axial_DIN0309_L9.0mm_D3.2mm_P12.70mm_Horizontal -> (none)
- R7: value 10 -> R; footprint Resistor_THT:R_Axial_DIN0309_L9.0mm_D3.2mm_P12.70mm_Horizontal -> (none)
- RSET7SEG1, RSETLED1: value 47k -> R_Small; footprint SamacSys_Parts:RESC2012X60N -> Resistor_THT:R_Axial_DIN0309_L9.0mm_D3.2mm_P12.70mm_Horizontal
- Speaker+1, Speaker-1: footprint MountingHole:MountingHole_2.5mm_Pad -> (none)
- U2: footprint SamacSys_Parts:SOP65P490X110-8N -> (none)
Connections:
- net labels added: DAC_IN
- net labels removed: DAC_OUT, SPI3_MISO
- wire segments 301 -> 261
- no-connect marks 3 -> 1
Other:
- moved on the sheet: 5V1, GND1
