File: Main_Board/_autosave-Main_Board.sch (KiCad schematic (older format))
At the start: 68 parts, among them IC1 AZ1085CD-3.3TRG1, J1 PJ-037A, U1 STM32L152ZCTx, U2 LM386, Y1 ABM10W-16.0000MHZ-4-B1U-T3

Commit message: Schem Pictures
Other:
- note added: "Speaker Circuit"
- note removed: "Hall Out Values"
- moved on the sheet: 5VOut1, BL1, BR1, C11, C24, C25, GPIOHeader1, J1, R8, TL1, TR1, Y1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
