File: Main_Board/Main_Board.sch (KiCad schematic (older format))
At the start: 74 parts, among them U1 STM32L152ZCTx, U2 LM386

Commit message: Updated Mainboard
Parts:
- removed 5V-3V3: ZLDO1117K33TC, TO-252_1, symbol SamacSys_Parts:ZLDO1117K33TC
- removed C11: 100n, SamacSys_Parts:CAPC1005X55N, symbol Device:C
- removed Crst0: C, Capacitor_SMD:C_1812_4532Metric_Pad1.57x3.40mm_HandSolder, symbol Device:C
- removed HALLOUT1, HALLSEL[0]1, HALLSEL[1]1, HALLSEL[2]1, UART_Rx1, UART_Tx1: MountingHole_Pad, MountingHole:MountingHole_2.7mm_Pad, symbol Mechanical:MountingHole_Pad
- removed R1: R_Small, Resistor_THT:R_Axial_DIN0309_L9.0mm_D3.2mm_P12.70mm_Horizontal, symbol Device:R_Small
- removed SEG0_7SEG1, SEG0_LED1, SEG1_7SEG1, SEG1_LED1, SEG2_7SEG1, SEG2_LED1, SEG3_7SEG1, SEG3_LED1, SEG4_7SEG1, SEG4_LED1, SEG5_7SEG1, SEG5_LED1, SEG6_7SEG1, SEG6_LED1, SEG7_7SEG1, SEG7_LED1, SEG8_7SEG1, SEG8_LED1: MountingHole_Pad, MountingHole:MountingHole_2.5mm_Pad, symbol Mechanical:MountingHole_Pad
- removed nRST1: SW_MEC_5G, Button_Switch_SMD:Panasonic_EVQPUL_EVQPUC, symbol Switch:SW_MEC_5G
- added C17, C20: 22u, symbol Device:C_Small
- added C18, C19: 100n, SamacSys_Parts:CAPC2012X95N, symbol Device:C_Small
- added C21: C_Small, symbol Device:C_Small
- added C22: 10u, symbol Device:C
- added C23: 22u, symbol Device:C
- added HallSensorHeader1: Conn_01x04_Male, Connector_PinHeader_2.54mm:PinHeader_1x04_P2.54mm_Vertical, symbol Connector:Conn_01x04_Male
- added IC1: AZ1085CD-3.3TRG1, AZ1085CD33TRG1, symbol SamacSys_Parts:AZ1085CD-3.3TRG1
- added LED_Header1, LED_Header2: Conn_01x09_Male, Connector_PinHeader_2.54mm:PinHeader_1x09_P2.54mm_Vertical, symbol Connector:Conn_01x09_Male
- added SD_CARD1: 47352-1001, 47352-1001, symbol SamacSys_Parts:47352-1001
- added UARTHeader1: Conn_01x02_Male, Connector_PinHeader_2.54mm:PinHeader_1x02_P2.54mm_Vertical, symbol Connector:Conn_01x02_Male
- C0, C1, C10, C2, C3, C4, C5, C6, C7, C8, C9: footprint SamacSys_Parts:CAPC1005X55N -> SamacSys_Parts:CAPC2012X95N
- C12, C14, C15: footprint (none) -> SamacSys_Parts:CAPC2012X95N
- C13: footprint (none) -> SamacSys_Parts:CAPC2012X140N
- C16: footprint (none) -> Capacitor_THT:CP_Radial_D4.0mm_P2.00mm
- CA1: footprint SamacSys_Parts:CAPC1005X55N -> SamacSys_Parts:CAPC2012X140N
- CSET7SEG1, CSETLED1: value C_Small -> 47p; footprint Capacitor_SMD:C_1812_4532Metric_Pad1.57x3.40mm_HandSolder -> SamacSys_Parts:CAPC2012X75N
- R4, R5, R6: footprint (none) -> Resistor_THT:R_Axial_DIN0309_L9.0mm_D3.2mm_P12.70mm_Horizontal
- R7: value R -> 10; footprint (none) -> Resistor_THT:R_Axial_DIN0309_L9.0mm_D3.2mm_P12.70mm_Horizontal
- RSET7SEG1, RSETLED1: value R_Small -> 47k; footprint Resistor_THT:R_Axial_DIN0309_L9.0mm_D3.2mm_P12.70mm_Horizontal -> SamacSys_Parts:RESC2012X60N
- Speaker+1, Speaker-1: footprint (none) -> MountingHole:MountingHole_2.5mm_Pad
- U2: footprint (none) -> SamacSys_Parts:SOP65P490X110-8N
Connections:
- net labels added: DAC_OUT, SPI3_MISO
- net labels removed: DAC_IN
- wire segments 261 -> 301
- no-connect marks 1 -> 3
Other:
- moved on the sheet: 5V1, GND1

Commit message: A
Parts:
- added C11, C24: 30p, Capacitor_SMD:C_1206_3216Metric_Pad1.33x1.80mm_HandSolder, symbol Device:C
- added R1: 1M, SamacSys_Parts:RESC5025X70N, symbol Device:R
- added Y1: Crystal, Crystal:Crystal_HC18-U_Vertical, symbol Device:Crystal
- C17, C20: footprint (none) -> SamacSys_Parts:CAPC2012X95N
- JTAGHEADER1: footprint Connector_PinHeader_2.00mm:PinHeader_2x05_P2.00mm_Vertical -> Connector_PinHeader_2.54mm:PinHeader_2x05_P2.54mm_Vertical
- R4: footprint Resistor_THT:R_Axial_DIN0309_L9.0mm_D3.2mm_P12.70mm_Horizontal -> SamacSys_Parts:CRGCQ2512F3K3
- R5: footprint Resistor_THT:R_Axial_DIN0309_L9.0mm_D3.2mm_P12.70mm_Horizontal -> SamacSys_Parts:ERJ1TRQF1R0U
- R6: footprint Resistor_THT:R_Axial_DIN0309_L9.0mm_D3.2mm_P12.70mm_Horizontal -> SamacSys_Parts:RESC5025X70N
Connections:
- net labels added: Boot, OSC_IN, OSC_OUT
- net labels removed: JTRST
- wire segments 301 -> 314
Changed lines of the file:
@@
 	0    -1   -1   0
 $EndComp
-Wire Wire Line
-	17000 4550 17000 3750
-Text Label 17000 4400 1    50   ~ 0
-JTRST
 Text GLabel 16200 3750 1    50   Input ~ 0
 JTMS-SWDIO
@@
 Text GLabel 16900 3750 1    50   Input ~ 0
 JTDO-SWO
-Text GLabel 17000 3750 1    50   Input ~ 0
-JTRST
 Wire Wire Line
 	15800 4550 15800 3900
@@
 LED Driver Circuit
 $Comp
-L SamacSys_Parts:MAX6951CEE+ 7SEGDriver1
-U 1 1 616F30CA
-P 6350 3400
-F 0 "7SEGDriver1" H 7250 3400 50  0000 C CNN
-F 1 "MAX6951CEE+" H 7250 2650 50  0000 C CNN
-F 2 "SOP64P602X173-17N" H 8000 3500 50  0001 L CNN
-F 3 "https://datasheets.maximintegrated.com/en/ds/MAX6950-MAX6951.pdf" H 8000 3400 50  0001 L CNN
-F 4 "LED Driver 64Segment 3.3V/5V" H 8000 3300 50  0001 L CNN "Description"
-F 5 "1.73" H 8000 3200 50  0001 L CNN "Height"
-F 6 "700-MAX6951CEE" H 8000 3100 50  0001 L CNN "Mouser Part Number"
-F 7 "https://www.mouser.co.uk/ProductDetail/Maxim-Integrated/MAX6951CEE%2b?qs=1THa7WoU59G039lytpTsUQ%3D%3D" H 8000 3000 50  0001 L CNN "Mouser Price/Stock"
-F 8 "Maxim Integrated" H 8000 2900 50  0001 L CNN "Manufacturer_Name"
-F 9 "MAX6951CEE+" H 8000 2800 50  0001 L CNN "Manufacturer_Part_Number"
-	1    6350 3400
-	1    0    0    -1
-$EndComp
-$Comp
 L Device:R_Small RSET7SEG1
 U 1 1 616F30D0
@@
 F 0 "JTAGHEADER1" H 10450 3917 50  0000 C CNN
 F 1 "Conn_02x05_Odd_Even" H 10450 3826 50  0000 C CNN
-F 2 "Connector_PinHeader_2.00mm:PinHeader_2x05_P2.00mm_Vertical" H 10400 3500 50  0001 C CNN
+F 2 "Connector_PinHeader_2.54mm:PinHeader_2x05_P2.54mm_Vertical" H 10400 3500 50  0001 C CNN
 F 3 "~" H 10400 3500 50  0001 C CNN
 	1    10400 3500
@@
 Wire Notes Line
 	13550 2250 13550 9600
-Wire Wire Line
-	14250 8550 14250 6750
-Wire Wire Line
-	14300 6750 14900 6750
 $Comp
 L Mechanical:MountingHole_Pad TL1
@@
 F 0 "R4" V 9093 8600 50  0000 C CNN
 F 1 "3300" V 9184 8600 50  0000 C CNN
-F 2 "Resistor_THT:R_Axial_DIN0309_L9.0mm_D3.2mm_P12.70mm_Horizontal" V 9230 8600 50  0001 C CNN
+F 2 "SamacSys_Parts:CRGCQ2512F3K3" V 9230 8600 50  0001 C CNN
 F 3 "~" H 9300 8600 50  0001 C CNN
 	1    9300 8600
@@
 F 0 "R5" H 9620 8846 50  0000 L CNN
 F 1 "150" H 9620 8755 50  0000 L CNN
-F 2 "Resistor_THT:R_Axial_DIN0309_L9.0mm_D3.2mm_P12.70mm_Horizontal" V 9480 8800 50  0001 C CNN
+F 2 "SamacSys_Parts:ERJ1TRQF1R0U" V 9480 8800 50  0001 C CNN
 F 3 "~" H 9550 8800 50  0001 C CNN
 	1    9550 8800
@@
 F 0 "R6" V 9643 8600 50  0000 C CNN
 F 1 "100" V 9734 8600 50  0000 C CNN
-F 2 "Resistor_THT:R_Axial_DIN0309_L9.0mm_D3.2mm_P12.70mm_Horizontal" V 9780 8600 50  0001 C CNN
+F 2 "SamacSys_Parts:RESC5025X70N" V 9780 8600 50  0001 C CNN
 F 3 "~" H 9850 8600 50  0001 C CNN
 	1    9850 8600
@@
 F 0 "C17" H 4092 3346 50  0000 L CNN
 F 1 "22u" H 4092 3255 50  0000 L CNN
-F 2 "" H 4000 3300 50  0001 C CNN
+F 2 "SamacSys_Parts:CAPC2012X95N" H 4000 3300 50  0001 C CNN
 F 3 "~" H 4000 3300 50  0001 C CNN
 	1    4000 3300
@@
 F 0 "C20" H 8442 3346 50  0000 L CNN
 F 1 "22u" H 8442 3255 50  0000 L CNN
-F 2 "" H 8350 3300 50  0001 C CNN
+F 2 "SamacSys_Parts:CAPC2012X95N" H 8350 3300 50  0001 C CNN
 F 3 "~" H 8350 3300 50  0001 C CNN
 	1    8350 3300
@@
 Wire Wire Line
 	8450 3400 8350 3400
-Connection ~ 8150 3400
 Connection ~ 8350 3400
 Wire Wire Line
@@
 	6700 3050 6700 2700
 Wire Wire Line
-	5850 2950 5850 3600
-Wire Wire Line
-	5750 2900 5750 3700
-Wire Wire Line
-	5650 2850 5650 3800
-Wire Wire Line
 	5550 2800 5550 3900
 Wire Wire Line
@@
 Wire Wire Line
 	11150 6600 11150 6450
+Text GLabel 14900 6750 3    50   Input ~ 0
+nRST
+$Comp
+L Device:Crystal Y1
+U 1 1 61878275
+P 16250 7200
+F 0 "Y1" H 16250 7468 50  0000 C CNN
+F 1 "Crystal" H 16250 7377 50  0000 C CNN
+F 2 "Crystal:Crystal_HC18-U_Vertical" H 16250 7200 50  0001 C CNN
+F 3 "~" H 16250 7200 50  0001 C CNN
+	1    16250 7200
+	1    0    0    -1
+$EndComp
+$Comp
+L Device:C C24
+U 1 1 6187994F
+P 16550 7350
+F 0 "C24" H 16665 7396 50  0000 L CNN
+F 1 "30p" H 16665 7305 50  0000 L CNN
+F 2 "Capacitor_SMD:C_1206_3216Metric_Pad1.33x1.80mm_HandSolder" H 16588 7200 50  0001 C CNN
+F 3 "~" H 16550 7350 50  0001 C CNN
+	1    16550 7350
+	1    0    0    -1
+$EndComp
+$Comp
+L Device:C C11
+U 1 1 6187AF45
+P 15900 7350
+F 0 "C11" H 16015 7396 50  0000 L CNN
+F 1 "30p" H 16015 7305 50  0000 L CNN
+F 2 "Capacitor_SMD:C_1206_3216Metric_Pad1.33x1.80mm_HandSolder" H 15938 7200 50  0001 C CNN
+F 3 "~" H 15900 7350 50  0001 C CNN
+	1    15900 7350
+	1    0    0    -1
+$EndComp
+$Comp
+L power:GND #PWR0118
+U 1 1 6187B618
+P 16250 7600
+F 0 "#PWR0118" H 16250 7350 50  0001 C CNN
+F 1 "GND" H 16255 7427 50  0000 C CNN
+F 2 "" H 16250 7600 50  0001 C CNN
+F 3 "" H 16250 7600 50  0001 C CNN
+	1    16250 7600
+	1    0    0    -1
+$EndComp
+Wire Wire Line
+	16550 7500 16250 7500
+Wire Wire Line
+	16250 7500 16250 7600
+Wire Wire Line
+	15900 7500 16250 7500
+Connection ~ 16250 7500
+Wire Wire Line
+	15900 7200 16100 7200
+Wire Wire Line
+	16400 7200 16550 7200
+Wire Wire Line
+	16200 6750 16200 6800
+Wire Wire Line
+	16200 6800 15900 6800
+Wire Wire Line
+	15900 6800 15900 6900
+Connection ~ 15900 7200
+Wire Wire Line
+	16300 6750 16300 6800
+Wire Wire Line
+	16300 6800 16550 6800
+Wire Wire Line
+	16550 6800 16550 6900
+Connection ~ 16550 7200
+Text Label 15900 6800 0    50   ~ 0
+OSC_IN
+Text Label 16350 6800 0    50   ~ 0
+OSC_OUT
+$Comp
+L Device:R R1
+U 1 1 61922B72
+P 16250 6900
+F 0 "R1" V 16043 6900 50  0000 C CNN
+F 1 "1M" V 16134 6900 50  0000 C CNN
+F 2 "SamacSys_Parts:RESC5025X70N" V 16180 6900 50  0001 C CNN
+F 3 "~" H 16250 6900 50  0001 C CNN
+	1    16250 6900
+	0    1    1    0
+$EndComp
+Wire Wire Line
+	16400 6900 16550 6900
+Connection ~ 16550 6900
+Wire Wire Line
+	16550 6900 16550 7200
+Wire Wire Line
+	16100 6900 15900 6900
+Connection ~ 15900 6900
+Wire Wire Line
+	15900 6900 15900 7200
+Wire Wire Line
+	15100 6750 15100 7000
+Text GLabel 15100 7000 3    50   Input ~ 0
+Boot
+Text Label 15100 6900 0    50   ~ 0
+Boot
+Connection ~ 8150 3400
+Wire Wire Line
+	5650 2850 5650 3800
+Wire Wire Line
+	5750 2900 5750 3700
+Wire Wire Line
+	5850 2950 5850 3600
+$Comp
+L SamacSys_Parts:MAX6951CEE+ 7SEGDriver1
+U 1 1 616F30CA
+P 6350 3400
+F 0 "7SEGDriver1" H 7250 3400 50  0000 C CNN
+F 1 "MAX6951CEE+" H 7250 2650 50  0000 C CNN
+F 2 "SOP64P602X173-17N" H 8000 3500 50  0001 L CNN
+F 3 "https://datasheets.maximintegrated.com/en/ds/MAX6950-MAX6951.pdf" H 8000 3400 50  0001 L CNN
+F 4 "LED Driver 64Segment 3.3V/5V" H 8000 3300 50  0001 L CNN "Description"
+F 5 "1.73" H 8000 3200 50  0001 L CNN "Height"
+F 6 "700-MAX6951CEE" H 8000 3100 50  0001 L CNN "Mouser Part Number"
+F 7 "https://www.mouser.co.uk/ProductDetail/Maxim-Integrated/MAX6951CEE%2b?qs=1THa7WoU59G039lytpTsUQ%3D%3D" H 8000 3000 50  0001 L CNN "Mouser Price/Stock"
+F 8 "Maxim Integrated" H 8000 2900 50  0001 L CNN "Manufacturer_Name"
+F 9 "MAX6951CEE+" H 8000 2800 50  0001 L CNN "Manufacturer_Part_Number"
+	1    6350 3400
+	1    0    0    -1
+$EndComp
 $EndSCHEMATC

Commit message: Added switch board, reset circuit
Parts:
- added C25: 0.1u, symbol Device:C
- added R8: 10k, symbol Device:R
- added S1: PTS647SM50SMTR2LFS, Main_Board:PTS647SM50SMTR2LFS, symbol rst_button:PTS647SM50SMTR2LFS
- 7SEGDriver1, LEDDriver1: symbol SamacSys_Parts:MAX6951CEE+ -> Main_Board-rescue:MAX6951CEE+-SamacSys_Parts
- IC1: symbol SamacSys_Parts:AZ1085CD-3.3TRG1 -> Main_Board-rescue:AZ1085CD-3.3TRG1-SamacSys_Parts
- LED3V3, LED5V1: symbol xzcfbb53w-8vf:XZCFBB53W-8VF -> Main_Board-rescue:XZCFBB53W-8VF-xzcfbb53w-8vf
- SD_CARD1: symbol SamacSys_Parts:47352-1001 -> Main_Board-rescue:47352-1001-SamacSys_Parts
Connections:
- net labels removed: Boot
- wire segments 314 -> 325
Changed lines of the file:
@@
 $EndComp
 $Comp
-L xzcfbb53w-8vf:XZCFBB53W-8VF LED5V1
+L Main_Board-rescue:XZCFBB53W-8VF-xzcfbb53w-8vf LED5V1
 U 1 1 614E1141
 P 21900 10700
@@
 $EndComp
 $Comp
-L xzcfbb53w-8vf:XZCFBB53W-8VF LED3V3
+L Main_Board-rescue:XZCFBB53W-8VF-xzcfbb53w-8vf LED3V3
 U 1 1 614E1E21
 P 22400 10700
@@
 $EndComp
 $Comp
-L SamacSys_Parts:MAX6951CEE+ LEDDriver1
+L Main_Board-rescue:MAX6951CEE+-SamacSys_Parts LEDDriver1
 U 1 1 6164861C
 P 2200 3400
@@
 $EndComp
 $Comp
-L SamacSys_Parts:AZ1085CD-3.3TRG1 IC1
+L Main_Board-rescue:AZ1085CD-3.3TRG1-SamacSys_Parts IC1
 U 1 1 6187B1FB
 P 11450 5350
@@
 	6000 7150 13550 7150
 $Comp
-L SamacSys_Parts:47352-1001 SD_CARD1
+L Main_Board-rescue:47352-1001-SamacSys_Parts SD_CARD1
 U 1 1 6161C0A1
 P 6450 6300
@@
 	15900 6900 15900 7200
 Wire Wire Line
-	15100 6750 15100 7000
-Text GLabel 15100 7000 3    50   Input ~ 0
-Boot
-Text Label 15100 6900 0    50   ~ 0
-Boot
+	15100 6750 15100 6950
 Connection ~ 8150 3400
 Wire Wire Line
@@
 	5850 2950 5850 3600
 $Comp
-L SamacSys_Parts:MAX6951CEE+ 7SEGDriver1
+L Main_Board-rescue:MAX6951CEE+-SamacSys_Parts 7SEGDriver1
 U 1 1 616F30CA
 P 6350 3400
@@
 	1    0    0    -1
 $EndComp
+$Comp
+L power:GND #PWR0123
+U 1 1 6167AAA4
+P 15100 6950
+F 0 "#PWR0123" H 15100 6700 50  0001 C CNN
+F 1 "GND" H 15105 6777 50  0000 C CNN
+F 2 "" H 15100 6950 50  0001 C CNN
+F 3 "" H 15100 6950 50  0001 C CNN
+	1    15100 6950
+	1    0    0    -1
+$EndComp
+Text GLabel 13850 8900 0    50   Input ~ 0
+nRST
+$Comp
+L Device:R R8
+U 1 1 61698FFF
+P 14100 8650
+F 0 "R8" H 14170 8696 50  0000 L CNN
+F 1 "10k" H 14170 8605 50  0000 L CNN
+F 2 "" V 14030 8650 50  0001 C CNN
+F 3 "~" H 14100 8650 50  0001 C CNN
+	1    14100 8650
+	1    0    0    -1
+$EndComp
+$Comp
+L power:+3V3 #PWR0124
+U 1 1 6169A4D6
+P 14100 8500
+F 0 "#PWR0124" H 14100 8350 50  0001 C CNN
+F 1 "+3V3" H 14115 8673 50  0000 C CNN
+F 2 "" H 14100 8500 50  0001 C CNN
+F 3 "" H 14100 8500 50  0001 C CNN
+	1    14100 8500
+	1    0    0    -1
+$EndComp
+$Comp
+L Device:C C25
+U 1 1 616B96CB
+P 14100 9150
+F 0 "C25" H 14215 9196 50  0000 L CNN
+F 1 "0.1u" H 14215 9105 50  0000 L CNN
+F 2 "" H 14138 9000 50  0001 C CNN
+F 3 "~" H 14100 9150 50  0001 C CNN
+	1    14100 9150
+	1    0    0    -1
+$EndComp
+$Comp
+L power:GND #PWR0127
+U 1 1 616BA68F
+P 14300 9350
+F 0 "#PWR0127" H 14300 9100 50  0001 C CNN
+F 1 "GND" H 14305 9177 50  0000 C CNN
+F 2 "" H 14300 9350 50  0001 C CNN
+F 3 "" H 14300 9350 50  0001 C CNN
+	1    14300 9350
+	1    0    0    -1
+$EndComp
+$Comp
+L rst_button:PTS647SM50SMTR2LFS S1
+U 1 1 616BD552
+P 14750 8550
+F 0 "S1" V 15104 8678 50  0000 L CNN
+F 1 "PTS647SM50SMTR2LFS" V 15195 8678 50  0000 L CNN
+F 2 "Main_Board:PTS647SM50SMTR2LFS" H 15400 8650 50  0001 L CNN
+F 3 "https://www.ckswitches.com/media/2567/pts647.pdf" H 15400 8550 50  0001 L CNN
+F 4 "Tactile Switches 50mA 12VDC, 1.8N 5.0mm H, G leads" H 15400 8450 50  0001 L CNN "Description"
+F 5 "5.25" H 15400 8350 50  0001 L CNN "Height"
+F 6 "611-PTS647SM50SMTR2L" H 15400 8250 50  0001 L CNN "Mouser Part Number"
+F 7 "https://www.mouser.co.uk/ProductDetail/CK/PTS647SM50SMTR2LFS?qs=PqoDHHvF64%252BjK4ZB7f42kw%3D%3D" H 15400 8150 50  0001 L CNN "Mouser Price/Stock"
+F 8 "C & K COMPONENTS" H 15400 8050 50  0001 L CNN "Manufacturer_Name"
+F 9 "PTS647SM50SMTR2LFS" H 15400 7950 50  0001 L CNN "Manufacturer_Part_Number"
+	1    14750 8550
+	0    1    1    0
+$EndComp
+Wire Wire Line
+	13850 8900 14100 8900
+Wire Wire Line
+	14100 8900 14100 9000
+Wire Wire Line
+	14100 8900 14100 8800
+Connection ~ 14100 8900
+Wire Wire Line
+	14100 8900 14450 8900
+Wire Wire Line
+	14450 8900 14450 8550
+Wire Wire Line
+	14450 8550 14650 8550
+Wire Wire Line
+	14750 8550 14650 8550
+Connection ~ 14650 8550
+Wire Wire Line
+	14750 9350 14650 9350
+Wire Wire Line
+	14300 9350 14650 9350
+Connection ~ 14650 9350
+Wire Wire Line
+	14300 9350 14100 9350
+Wire Wire Line
+	14100 9350 14100 9300
+Connection ~ 14300 9350
 $EndSCHEMATC

Commit message: 8 Hall Sensor
Parts:
- removed C25: 0.1u, symbol Device:C
- removed HallSensorHeader1: Conn_01x04_Male, Connector_PinHeader_2.54mm:PinHeader_1x04_P2.54mm_Vertical, symbol Connector:Conn_01x04_Male
- removed R8: 10k, symbol Device:R
- removed S1: PTS647SM50SMTR2LFS, Main_Board:PTS647SM50SMTR2LFS, symbol rst_button:PTS647SM50SMTR2LFS
- added C25: C_Small, SamacSys_Parts:CAPC2012X140N, symbol Device:C_Small
- added J1: Conn_01x08, Connector_PinHeader_2.54mm:PinHeader_1x08_P2.54mm_Vertical, symbol Connector_Generic:Conn_01x08
- added J2: Conn_01x03_Male, Connector_PinHeader_2.54mm:PinHeader_1x03_P2.54mm_Vertical, symbol Connector:Conn_01x03_Male
- added R8: R_Small, SamacSys_Parts:RESC5025X70N, symbol Device:R_Small
- added e1: SW_MEC_5G, Button_Switch_SMD:SW_SPST_Omron_B3FS-105xP, symbol Switch:SW_MEC_5G
- 7SEGDriver1, LEDDriver1: symbol Main_Board-rescue:MAX6951CEE+-SamacSys_Parts -> SamacSys_Parts:MAX6951CEE+
- IC1: symbol Main_Board-rescue:AZ1085CD-3.3TRG1-SamacSys_Parts -> SamacSys_Parts:AZ1085CD-3.3TRG1
- LED3V3, LED5V1: symbol Main_Board-rescue:XZCFBB53W-8VF-xzcfbb53w-8vf -> xzcfbb53w-8vf:XZCFBB53W-8VF
- SD_CARD1: symbol Main_Board-rescue:47352-1001-SamacSys_Parts -> SamacSys_Parts:47352-1001
Connections:
- net labels added: Boot, HALLOUT[0], HALLOUT[1], HALLOUT[2], HALLOUT[3], HALLOUT[4], HALLOUT[5], HALLOUT[6], HALLOUT[7]
- net labels removed: HALLOUT
- wire segments 325 -> 343
Other:
- note added: "Hall Out Values"
- note added: "Hall Sensor Select Circuitry\n"
- note removed: "Hall Sensor Circuitry\n"
- moved on the sheet: C11, C24, R1

Commit message: ''Updates 12-10"
Parts:
- removed C11, C24: 30p, Capacitor_SMD:C_1206_3216Metric_Pad1.33x1.80mm_HandSolder, symbol Device:C
- removed C16: 250u, Capacitor_THT:CP_Radial_D4.0mm_P2.00mm, symbol Device:C
- removed LED3V3: 3V3, LED Lib:XCXZCFBB53W-8VF, symbol xzcfbb53w-8vf:XZCFBB53W-8VF
- removed R1: 1M, SamacSys_Parts:RESC5025X70N, symbol Device:R
- removed R2, R3: R, Resistor_THT:R_Axial_DIN0309_L9.0mm_D3.2mm_P12.70mm_Horizontal, symbol Device:R
- removed R7: 10, Resistor_THT:R_Axial_DIN0309_L9.0mm_D3.2mm_P12.70mm_Horizontal, symbol Device:R
- removed Y1: Crystal, Crystal:Crystal_HC18-U_Vertical, symbol Device:Crystal
- removed e1: SW_MEC_5G, Button_Switch_SMD:SW_SPST_Omron_B3FS-105xP, symbol Switch:SW_MEC_5G
- added 5VOut1: Conn_01x02, Connector_PinHeader_2.54mm:PinHeader_1x02_P2.54mm_Vertical, symbol Connector_Generic:Conn_01x02
- added C11, C24: 4p, CAPC1005X55N, symbol SamacSys_Parts:GCQ1555C1H4R0CB01D
- added C16: 220u, CAPPRD200W55D500H1200, symbol SamacSys_Parts:ECA-0JHG221B
- added GPIOHeader1: Conn_01x09, Connector_PinHeader_2.54mm:PinHeader_1x09_P2.54mm_Vertical, symbol Connector_Generic:Conn_01x09
- added LED3V3: 3V3, LEDM168X65N, symbol SamacSys_Parts:SMLD12BN1WT86
- added R2: 680, RESC3116X70N, symbol SamacSys_Parts:ERJ-UP8F6800V
- added R3: 82, RESC6432X65N, symbol SamacSys_Parts:CRGP2512F82R
- added R7: 10, RESC5025X120N, symbol SamacSys_Parts:350210RFT
- added Y1: ABM10W-16.0000MHZ-4-B1U-T3, ABM10W400000MHZ4K1ZT3, symbol SamacSys_Parts:ABM10W-16.0000MHZ-4-B1U-T3
- added nRST1: PTS647SM50SMTR2LFS, PTS647SM50SMTR2LFS, symbol SamacSys_Parts:PTS647SM50SMTR2LFS
- C17, C20: footprint SamacSys_Parts:CAPC2012X95N -> SamacSys_Parts:C1608_Commercial
- C21: value C_Small -> 1u; footprint (none) -> SamacSys_Parts:CAPC1005X55N
- C22: footprint (none) -> SamacSys_Parts:CAPC2012X140N
- C23: footprint (none) -> SamacSys_Parts:C1608_Commercial
- C25: value C_Small -> 100n; footprint SamacSys_Parts:CAPC2012X140N -> SamacSys_Parts:CAPC2012X95N
- CA1: footprint SamacSys_Parts:CAPC2012X140N -> SamacSys_Parts:CAPC0402X22N
- LA0: footprint Inductor_SMD:L_01005_0402Metric_Pad0.57x0.30mm_HandSolder -> SamacSys_Parts:LQW2UAS12NG00L
- LED5V1: footprint LED Lib:XCXZCFBB53W-8VF -> SamacSys_Parts:HSMA-C380
- R8: value R_Small -> 10k; footprint SamacSys_Parts:RESC5025X70N -> SamacSys_Parts:RESC3116X70N
- renumbered LED_Header2 to 7_Seg_Header1, J1 to Hal_Out_Header1, J2 to Hall_Sel_Header1
Connections:
- net labels added: S1[1], S1[2], S1[3], S2[1], S2[2], S2[3]
- wire segments 343 -> 371
Other:
- note added: "Crystal Circuitry"
- note added: "Debug LEDs"
- note added: "GPIO Header"
- moved on the sheet: Speaker+1

Commit message: fixed reverse biased LEDs
Parts:
- 7SEGDriver1, LEDDriver1: symbol SamacSys_Parts:MAX6951CEE+ -> Main_Board-rescue:MAX6951CEE+-SamacSys_Parts
- C11, C24: symbol SamacSys_Parts:GCQ1555C1H4R0CB01D -> Main_Board-rescue:GCQ1555C1H4R0CB01D-SamacSys_Parts
- C16: symbol SamacSys_Parts:ECA-0JHG221B -> Main_Board-rescue:ECA-0JHG221B-SamacSys_Parts
- IC1: symbol SamacSys_Parts:AZ1085CD-3.3TRG1 -> Main_Board-rescue:AZ1085CD-3.3TRG1-SamacSys_Parts
- LED3V3: symbol SamacSys_Parts:SMLD12BN1WT86 -> Main_Board-rescue:SMLD12BN1WT86-SamacSys_Parts
- LED5V1: symbol xzcfbb53w-8vf:XZCFBB53W-8VF -> Main_Board-rescue:XZCFBB53W-8VF-xzcfbb53w-8vf
- R2: symbol SamacSys_Parts:ERJ-UP8F6800V -> Main_Board-rescue:ERJ-UP8F6800V-SamacSys_Parts
- R3: symbol SamacSys_Parts:CRGP2512F82R -> Main_Board-rescue:CRGP2512F82R-SamacSys_Parts
- R7: symbol SamacSys_Parts:350210RFT -> Main_Board-rescue:350210RFT-SamacSys_Parts
- SD_CARD1: symbol SamacSys_Parts:47352-1001 -> Main_Board-rescue:47352-1001-SamacSys_Parts
- Y1: symbol SamacSys_Parts:ABM10W-16.0000MHZ-4-B1U-T3 -> Main_Board-rescue:ABM10W-16.0000MHZ-4-B1U-T3-SamacSys_Parts
- nRST1: symbol SamacSys_Parts:PTS647SM50SMTR2LFS -> Main_Board-rescue:PTS647SM50SMTR2LFS-SamacSys_Parts
Changed lines of the file:
@@
 $EndComp
 $Comp
-L xzcfbb53w-8vf:XZCFBB53W-8VF LED5V1
+L Main_Board-rescue:XZCFBB53W-8VF-xzcfbb53w-8vf LED5V1
 U 1 1 614E1141
 P 3500 5800
@@
 $EndComp
 $Comp
-L SamacSys_Parts:MAX6951CEE+ LEDDriver1
+L Main_Board-rescue:MAX6951CEE+-SamacSys_Parts LEDDriver1
 U 1 1 6164861C
 P 2200 3400
@@
 $EndComp
 $Comp
-L SamacSys_Parts:AZ1085CD-3.3TRG1 IC1
+L Main_Board-rescue:AZ1085CD-3.3TRG1-SamacSys_Parts IC1
 U 1 1 6187B1FB
 P 11450 5350
@@
 	7850 3250 6300 3250
 $Comp
-L SamacSys_Parts:47352-1001 SD_CARD1
+L Main_Board-rescue:47352-1001-SamacSys_Parts SD_CARD1
 U 1 1 6161C0A1
 P 6450 6300
@@
 	5850 2950 5850 3600
 $Comp
-L SamacSys_Parts:MAX6951CEE+ 7SEGDriver1
+L Main_Board-rescue:MAX6951CEE+-SamacSys_Parts 7SEGDriver1
 U 1 1 616F30CA
 P 6350 3400
@@
 GPIO Header
 $Comp
-L SamacSys_Parts:350210RFT R7
+L Main_Board-rescue:350210RFT-SamacSys_Parts R7
 U 1 1 6222D435
 P 11650 9050
@@
 	10850 9300 10850 9350
 $Comp
-L SamacSys_Parts:SMLD12BN1WT86 LED3V3
+L Main_Board-rescue:SMLD12BN1WT86-SamacSys_Parts LED3V3
 U 1 1 622EEDCF
 P 4700 6100
@@
 	8600 5800 8600 9850
 $Comp
-L SamacSys_Parts:CRGP2512F82R R3
+L Main_Board-rescue:CRGP2512F82R-SamacSys_Parts R3
 U 1 1 6259D6C6
 P 4700 6100
@@
 $EndComp
 $Comp
-L SamacSys_Parts:ERJ-UP8F6800V R2
+L Main_Board-rescue:ERJ-UP8F6800V-SamacSys_Parts R2
 U 1 1 62633D18
 P 3650 6050
@@
 	12450 8700 12400 8700
 $Comp
-L SamacSys_Parts:ECA-0JHG221B C16
+L Main_Board-rescue:ECA-0JHG221B-SamacSys_Parts C16
 U 1 1 627085A6
 P 11900 8700
@@
 $EndComp
 $Comp
-L SamacSys_Parts:PTS647SM50SMTR2LFS nRST1
+L Main_Board-rescue:PTS647SM50SMTR2LFS-SamacSys_Parts nRST1
 U 1 1 627772E3
 P 14500 8900
@@
 	13900 9200 13900 9700
 $Comp
-L SamacSys_Parts:ABM10W-16.0000MHZ-4-B1U-T3 Y1
+L Main_Board-rescue:ABM10W-16.0000MHZ-4-B1U-T3-SamacSys_Parts Y1
 U 1 1 6281C654
 P 16900 8550
@@
 Connection ~ 17200 9300
 $Comp
-L SamacSys_Parts:GCQ1555C1H4R0CB01D C24
+L Main_Board-rescue:GCQ1555C1H4R0CB01D-SamacSys_Parts C24
 U 1 1 62B1EF4C
 P 17750 8750
@@
 $EndComp
 $Comp
-L SamacSys_Parts:GCQ1555C1H4R0CB01D C11
+L Main_Board-rescue:GCQ1555C1H4R0CB01D-SamacSys_Parts C11
 U 1 1 62B45D13
 P 16850 8750
