File: Main_Board/Main_Board.sch (KiCad schematic (older format))
At the start: 67 parts, among them IC1 AZ1085CD-3.3TRG1, U1 STM32L152ZCTx, U2 LM386, Y1 ABM10W-16.0000MHZ-4-B1U-T3

Commit message: added DC jack, miscellaneous
Parts:
- removed 5V1, GND1: MountingHole_Pad, MountingHole:MountingHole_4.3mm_M4_Pad, symbol Mechanical:MountingHole_Pad
- added J1: PJ-037A, Main_Board:PJ037A, symbol SamacSys_Parts:PJ-037A
- LEDDriver1: symbol Main_Board-rescue:MAX6951CEE+-SamacSys_Parts -> main_board_parts:MAX6951CEE+
Connections:
- net +5V: now also J1.1
- net GND: now also J1.2
Changed lines of the file:
@@
 5V->3V3\n
-$Comp
-L Mechanical:MountingHole_Pad 5V1
-U 1 1 616143BB
-P 10950 5600
-F 0 "5V1" H 10850 5557 50  0000 R CNN
-F 1 "MountingHole_Pad" H 10850 5648 50  0000 R CNN
-F 2 "MountingHole:MountingHole_4.3mm_M4_Pad" H 10950 5600 50  0001 C CNN
-F 3 "~" H 10950 5600 50  0001 C CNN
-	1    10950 5600
-	-1   0    0    1
-$EndComp
 $Comp
 L power:+3V3 #PWR0125
@@
 	1    0    0    -1
 $EndComp
-Connection ~ 10950 5300
-Connection ~ 10950 5500
 Text GLabel 9000 8600 0    50   Input ~ 0
 DAC_OUT
@@
 $EndComp
 $Comp
-L Main_Board-rescue:MAX6951CEE+-SamacSys_Parts LEDDriver1
+L main_board_parts:MAX6951CEE+ LEDDriver1
 U 1 1 6164861C
 P 2200 3400
@@
 Wire Wire Line
 	8950 5250 9300 5250
-$Comp
-L Mechanical:MountingHole_Pad GND1
-U 1 1 616136E7
-P 10950 5200
-F 0 "GND1" H 11050 5249 50  0000 L CNN
-F 1 "MountingHole_Pad" H 11200 5300 50  0000 L CNN
-F 2 "MountingHole:MountingHole_4.3mm_M4_Pad" H 10950 5200 50  0001 C CNN
-F 3 "~" H 10950 5200 50  0001 C CNN
-	1    10950 5200
-	1    0    0    -1
-$EndComp
 Wire Wire Line
 	6700 7600 6700 7550
@@
 $EndComp
 $Comp
-L power:+3.3VA #PWR?
+L power:+3.3VA #PWR0149
 U 1 1 6356791F
 P 15250 7450
-F 0 "#PWR?" H 15250 7300 50  0001 C CNN
+F 0 "#PWR0149" H 15250 7300 50  0001 C CNN
 F 1 "+3.3VA" H 15265 7623 50  0000 C CNN
 F 2 "" H 15250 7450 50  0001 C CNN
@@
 	-1   0    0    1
 $EndComp
+$Comp
+L SamacSys_Parts:PJ-037A J1
+U 1 1 6169B4AA
+P 4100 8550
+F 0 "J1" H 4728 8546 50  0000 L CNN
+F 1 "PJ-037A" H 4728 8455 50  0000 L CNN
+F 2 "Main_Board:PJ037A" H 4750 8650 50  0001 L CNN
+F 3 "" H 4750 8550 50  0001 L CNN
+F 4 "DC Power Connectors Power Jacks" H 4750 8450 50  0001 L CNN "Description"
+F 5 "11" H 4750 8350 50  0001 L CNN "Height"
+F 6 "490-PJ-037A" H 4750 8250 50  0001 L CNN "Mouser Part Number"
+F 7 "https://www.mouser.co.uk/ProductDetail/CUI-Devices/PJ-037A?qs=WyjlAZoYn53bdNRXfildEA%3D%3D" H 4750 8150 50  0001 L CNN "Mouser Price/Stock"
+F 8 "CUI Inc." H 4750 8050 50  0001 L CNN "Manufacturer_Name"
+F 9 "PJ-037A" H 4750 7950 50  0001 L CNN "Manufacturer_Part_Number"
+	1    4100 8550
+	1    0    0    -1
+$EndComp
+$Comp
+L power:GND #PWR0151
+U 1 1 6169E3BF
+P 4100 8550
+F 0 "#PWR0151" H 4100 8300 50  0001 C CNN
+F 1 "GND" V 4105 8422 50  0000 R CNN
+F 2 "" H 4100 8550 50  0001 C CNN
+F 3 "" H 4100 8550 50  0001 C CNN
+	1    4100 8550
+	0    1    1    0
+$EndComp
+$Comp
+L power:+5V #PWR0152
+U 1 1 6169F813
+P 4100 8650
+F 0 "#PWR0152" H 4100 8500 50  0001 C CNN
+F 1 "+5V" V 4115 8778 50  0000 L CNN
+F 2 "" H 4100 8650 50  0001 C CNN
+F 3 "" H 4100 8650 50  0001 C CNN
+	1    4100 8650
+	0    -1   -1   0
+$EndComp
 $EndSCHEMATC

Commit message: changed LM386 package to match what I bought
Parts:
- J1: symbol SamacSys_Parts:PJ-037A -> Main_Board-rescue:PJ-037A-SamacSys_Parts
- U2: footprint SamacSys_Parts:SOP65P490X110-8N -> SamacSys_Parts:SOIC127P600X175-8N
Changed lines of the file:
@@
 F 0 "U2" H 11294 8746 50  0000 L CNN
 F 1 "LM386" H 11294 8655 50  0000 L CNN
-F 2 "SamacSys_Parts:SOP65P490X110-8N" H 11050 8800 50  0001 C CNN
+F 2 "SamacSys_Parts:SOIC127P600X175-8N" H 11050 8800 50  0001 C CNN
 F 3 "http://www.ti.com/lit/ds/symlink/lm386.pdf" H 11150 8900 50  0001 C CNN
 	1    10950 8700
@@
 $EndComp
 $Comp
-L SamacSys_Parts:PJ-037A J1
+L Main_Board-rescue:PJ-037A-SamacSys_Parts J1
 U 1 1 6169B4AA
 P 4100 8550
