File: Main_Board/Main_Board.sch (KiCad schematic (older format))
At the start: 68 parts, among them IC1 AZ1085CD-3.3TRG1, J1 PJ-037A, U1 STM32L152ZCTx, U2 LM386, Y1 ABM10W-16.0000MHZ-4-B1U-T3

Commit message: edited main board headers for buttons, daughterboard power
Parts:
- removed GPIOHeader1: Conn_01x09, Connector_PinHeader_2.54mm:PinHeader_1x09_P2.54mm_Vertical, symbol Connector_Generic:Conn_01x09
- added DBoardPower1: Conn_01x02_Male, Main_Board:PinHeader_1x02_P2.54mm_Vertical, symbol Connector:Conn_01x02_Male
- added J2: 77311-862-11LF, HDRV11W62P0X254_1X11_2794X240X853P, symbol main_board_parts:77311-862-11LF
- UARTHeader1: footprint Connector_PinHeader_2.54mm:PinHeader_1x02_P2.54mm_Vertical -> Main_Board:PinHeader_1x02_P2.54mm_Vertical
Connections:
- net labels added: B1, B2
- net labels removed: Reset_Line
- wire segments 364 -> 360
- no-connect marks 85 -> 83
Other:
- note added: "Power Headers"
- note removed: "5V Headers"
Changed lines of the file:
@@
 F 0 "UARTHeader1" V 11312 6294 50  0000 L CNN
 F 1 "Conn_01x02_Male" V 11150 5700 50  0000 L CNN
-F 2 "Connector_PinHeader_2.54mm:PinHeader_1x02_P2.54mm_Vertical" H 11250 6250 50  0001 C CNN
+F 2 "Main_Board:PinHeader_1x02_P2.54mm_Vertical" H 11250 6250 50  0001 C CNN
 F 3 "~" H 11250 6250 50  0001 C CNN
 	1    11250 6250
@@
 Text Label 17400 7050 1    50   ~ 0
 S2[3]
-Text GLabel 1850 8800 3    50   Input ~ 0
+Text GLabel 1750 8650 3    50   Input ~ 0
 S1[1]
-Text GLabel 1950 8800 3    50   Input ~ 0
+Text GLabel 1850 8650 3    50   Input ~ 0
 S1[2]
-Text GLabel 2050 8800 3    50   Input ~ 0
+Text GLabel 1950 8650 3    50   Input ~ 0
 S1[3]
-Text GLabel 2150 8800 3    50   Input ~ 0
+Text GLabel 2050 8650 3    50   Input ~ 0
 S2[1]
-Text GLabel 2250 8800 3    50   Input ~ 0
+Text GLabel 2150 8650 3    50   Input ~ 0
 S2[2]
-Text GLabel 2350 8800 3    50   Input ~ 0
+Text GLabel 2250 8650 3    50   Input ~ 0
 S2[3]
-$Comp
-L Connector_Generic:Conn_01x09 GPIOHeader1
-U 1 1 61F622A8
-P 1950 8300
-F 0 "GPIOHeader1" V 2167 8296 50  0000 C CNN
-F 1 "Conn_01x09" V 2076 8296 50  0000 C CNN
-F 2 "Connector_PinHeader_2.54mm:PinHeader_1x09_P2.54mm_Vertical" H 1950 8300 50  0001 C CNN
-F 3 "~" H 1950 8300 50  0001 C CNN
-	1    1950 8300
-	0    -1   -1   0
-$EndComp
 $Comp
 L power:GND #PWR0128
 U 1 1 6200EDD4
-P 1550 8700
-F 0 "#PWR0128" H 1550 8450 50  0001 C CNN
-F 1 "GND" H 1555 8527 50  0000 C CNN
-F 2 "" H 1550 8700 50  0001 C CNN
-F 3 "" H 1550 8700 50  0001 C CNN
-	1    1550 8700
+P 2450 8350
+F 0 "#PWR0128" H 2450 8100 50  0001 C CNN
+F 1 "GND" H 2550 8200 50  0000 C CNN
+F 2 "" H 2450 8350 50  0001 C CNN
+F 3 "" H 2450 8350 50  0001 C CNN
+	1    2450 8350
 	1    0    0    -1
 $EndComp
@@
 L power:+3V3 #PWR0144
 U 1 1 62010503
-P 1700 8700
-F 0 "#PWR0144" H 1700 8550 50  0001 C CNN
-F 1 "+3V3" H 1715 8873 50  0000 C CNN
-F 2 "" H 1700 8700 50  0001 C CNN
-F 3 "" H 1700 8700 50  0001 C CNN
-	1    1700 8700
+P 2350 8350
+F 0 "#PWR0144" H 2350 8200 50  0001 C CNN
+F 1 "+3V3" H 2350 8500 50  0000 C CNN
+F 2 "" H 2350 8350 50  0001 C CNN
+F 3 "" H 2350 8350 50  0001 C CNN
+	1    2350 8350
 	-1   0    0    1
 $EndComp
-Wire Wire Line
-	1750 8650 1750 8500
-Wire Wire Line
-	1850 8800 1850 8500
-Wire Wire Line
-	1950 8800 1950 8500
-Wire Wire Line
-	2050 8800 2050 8500
-Wire Wire Line
-	2150 8800 2150 8500
-Wire Wire Line
-	2250 8800 2250 8500
-Wire Wire Line
-	2350 8800 2350 8500
 Text Notes 2450 7300 0    50   ~ 0
 GPIO Header
@@
 	16300 6750 16300 7300
 Wire Wire Line
-	17100 6750 17100 7150
-Wire Wire Line
-	19300 3750 19300 4550
-$Comp
-L MCU_ST_STM32L1:STM32L152ZCTx U1
-U 1 1 61411083
-P 18200 5650
-F 0 "U1" V 18250 9800 50  0000 L CNN
-F 1 "STM32L152ZCTx" V 18150 9450 50  0000 L CNN
-F 2 "Package_QFP:LQFP-144_20x20mm_P0.5mm" H 17300 2250 50  0001 R CNN
-F 3 "http://www.st.com/st-web-ui/static/active/en/resource/technical/document/datasheet/DM00111457.pdf" H 18200 5650 50  0001 C CNN
-	1    18200 5650
-	0    -1   -1   0
-$EndComp
-Wire Wire Line
 	16200 6750 16200 7300
 Text Notes 13000 2350 0    50   ~ 0
-5V Headers
+Power Headers
 Wire Wire Line
 	6350 4100 6050 4100
@@
 	1    0    0    -1
 $EndComp
-Wire Wire Line
-	1650 8700 1550 8700
-Wire Wire Line
-	1750 8650 1700 8650
-Wire Wire Line
-	1700 8650 1700 8700
 Wire Wire Line
 	2250 3200 3250 3200
@@
 Wire Notes Line
 	1000 10050 13550 10050
-Wire Wire Line
-	16800 6750 16800 7400
-Text GLabel 16800 7400 3    50   Input ~ 0
-Reset_Line
-Text Label 16800 6950 3    50   ~ 0
-Reset_Line
-Wire Wire Line
-	1650 8500 1650 8700
-Wire Wire Line
-	1550 8500 1550 8650
-Wire Wire Line
-	1550 8650 1400 8650
-Wire Wire Line
-	1400 8650 1400 8800
-Text GLabel 1400 8800 3    50   Input ~ 0
-Reset_Line
 $Comp
 L power:PWR_FLAG #FLG0101
@@
 NoConn ~ 18700 4550
 NoConn ~ 18800 4550
-NoConn ~ 18900 4550
-NoConn ~ 19000 4550
 NoConn ~ 19100 4550
 NoConn ~ 19200 4550
@@
 NoConn ~ 21000 4550
 NoConn ~ 21100 4550
-NoConn ~ 21200 4550
-NoConn ~ 21300 4550
 NoConn ~ 21400 4550
 NoConn ~ 21500 4550
@@
 	20000 4550 20000 3900
 NoConn ~ 17800 4550
-NoConn ~ 18100 4150
+$Comp
+L main_board_parts:77311-862-11LF J2
+U 1 1 6172F492
+P 1450 8350
+F 0 "J2" V 1788 7222 50  0000 R CNN
+F 1 "77311-862-11LF" V 1697 7222 50  0000 R CNN
+F 2 "HDRV11W62P0X254_1X11_2794X240X853P" H 2100 8450 50  0001 L CNN
+F 3 "" H 2100 8350 50  0001 L CNN
+F 4 "Headers & Wire Housings BERGSTIK" H 2100 8250 50  0001 L CNN "Description"
+F 5 "8.53" H 2100 8150 50  0001 L CNN "Height"
+F 6 "" H 2100 8050 50  0001 L CNN "Mouser Part Number"
+F 7 "" H 2100 7950 50  0001 L CNN "Mouser Price/Stock"
+F 8 "Amphenol" H 2100 7850 50  0001 L CNN "Manufacturer_Name"
+F 9 "77311-862-11LF" H 2100 7750 50  0001 L CNN "Manufacturer_Part_Number"
+	1    1450 8350
+	0    -1   -1   0
+$EndComp
+Text GLabel 1550 8650 3    50   Input ~ 0
+B1
+Text GLabel 1650 8650 3    50   Input ~ 0
+B2
+NoConn ~ 16800 6750
+Text GLabel 21200 3750 1    50   Input ~ 0
+B1
+Text GLabel 21300 3750 1    50   Input ~ 0
+B2
+Wire Wire Line
+	1450 8650 1450 8350
+Wire Wire Line
+	1550 8650 1550 8350
+Wire Wire Line
+	1650 8650 1650 8350
+Wire Wire Line
+	1750 8350 1750 8650
+Wire Wire Line
+	1850 8650 1850 8350
+Wire Wire Line
+	1950 8650 1950 8350
+Wire Wire Line
+	2050 8650 2050 8350
+Wire Wire Line
+	2150 8350 2150 8650
+Wire Wire Line
+	2250 8350 2250 8650
+Text GLabel 1450 8650 3    50   Input ~ 0
+nRST
+Wire Wire Line
+	17100 6750 17100 7150
+Wire Wire Line
+	19300 3750 19300 4550
+$Comp
+L MCU_ST_STM32L1:STM32L152ZCTx U1
+U 1 1 61411083
+P 18200 5650
+F 0 "U1" V 18250 9800 50  0000 L CNN
+F 1 "STM32L152ZCTx" V 18150 9450 50  0000 L CNN
+F 2 "Package_QFP:LQFP-144_20x20mm_P0.5mm" H 17300 2250 50  0001 R CNN
+F 3 "http://www.st.com/st-web-ui/static/active/en/resource/technical/document/datasheet/DM00111457.pdf" H 18200 5650 50  0001 C CNN
+	1    18200 5650
+	0    -1   -1   0
+$EndComp
+NoConn ~ 19000 4550
+NoConn ~ 18900 4550
+Wire Wire Line
+	21300 3750 21300 4550
+Wire Wire Line
+	21200 3750 21200 4550
+$Comp
+L Connector:Conn_01x02_Male DBoardPower1
+U 1 1 6172C583
+P 12500 4250
+F 0 "DBoardPower1" V 12562 4294 50  0000 L CNN
+F 1 "Conn_01x02_Male" V 12400 3700 50  0000 L CNN
+F 2 "Main_Board:PinHeader_1x02_P2.54mm_Vertical" H 12500 4250 50  0001 C CNN
+F 3 "~" H 12500 4250 50  0001 C CNN
+	1    12500 4250
+	0    1    1    0
+$EndComp
+$Comp
+L power:GND #PWR0135
+U 1 1 6172D4C6
+P 12500 4450
+F 0 "#PWR0135" H 12500 4200 50  0001 C CNN
+F 1 "GND" H 12600 4250 50  0000 C CNN
+F 2 "" H 12500 4450 50  0001 C CNN
+F 3 "" H 12500 4450 50  0001 C CNN
+	1    12500 4450
+	1    0    0    -1
+$EndComp
+$Comp
+L power:+3V3 #PWR0143
+U 1 1 6172DEE6
+P 12400 4450
+F 0 "#PWR0143" H 12400 4300 50  0001 C CNN
+F 1 "+3V3" H 12500 4650 50  0000 C CNN
+F 2 "" H 12400 4450 50  0001 C CNN
+F 3 "" H 12400 4450 50  0001 C CNN
+	1    12400 4450
+	-1   0    0    1
+$EndComp
 $EndSCHEMATC

Commit message: changed audio resistor value, same package
Parts:
- J1: symbol SamacSys_Parts:PJ-037A -> Main_Board-rescue:PJ-037A-SamacSys_Parts
- R4: value 3300 -> 560
Changed lines of the file:
@@
 P 9300 8600
 F 0 "R4" V 9093 8600 50  0000 C CNN
-F 1 "3300" V 9184 8600 50  0000 C CNN
+F 1 "560" V 9184 8600 50  0000 C CNN
 F 2 "SamacSys_Parts:CRGCQ2512F3K3" V 9230 8600 50  0001 C CNN
 F 3 "~" H 9300 8600 50  0001 C CNN
@@
 $EndComp
 $Comp
-L SamacSys_Parts:PJ-037A J1
+L Main_Board-rescue:PJ-037A-SamacSys_Parts J1
 U 1 1 6169B4AA
 P 12200 3700

Commit message: ESD and Pullups
Parts:
- added R10, R11, R12, R13, R14, R15, R16, R17, R9: 50k, RESC1005X40N, symbol SamacSys_Parts:CRCW040250K0FKED
- added R18, R19, R20: 10k, SamacSys_Parts:RESC3116X70N, symbol Device:R_Small
- J2: footprint HDRV11W62P0X254_1X11_2794X240X853P -> Main_Board:HDRV11W62P0X254_1X11_2794X240X853P
Connections:
- net +3V3: now also R18.1, R19.1, R20.2
- net B1: now also R10.1; no longer J2.2
- net B2: now also R11.1; no longer J2.3
- net S1[1]: now also R12.1; no longer J2.4
- net S1[2]: now also R13.1; no longer J2.5
- net S1[3]: now also R14.1; no longer J2.6
- net S2[1]: now also R15.1; no longer J2.7
- net S2[2]: now also R16.1; no longer J2.8
- net S2[3]: now also R17.1; no longer J2.9
- net SPI3_NSS: now also R18.2
- net nRST: now also R9.1; no longer J2.1
- net at SD_CARD1.1 (DATA2): now also R19.2
- net at SD_CARD1.8 (DATA1): now also R20.1
- new net: J2.1, R9.2
- new net: J2.2, R10.2
- new net: J2.3, R11.2
- new net: J2.4, R12.2
- new net: J2.5, R13.2
- new net: J2.6, R14.2
- new net: J2.7, R15.2
- new net: J2.8, R16.2
- new net: J2.9, R17.2
- no-connect marks 83 -> 81
Other:
- moved on the sheet: J2

Commit message: new main board gerbers
Parts:
- R10, R11, R12, R13, R14, R15, R16, R17, R9: symbol SamacSys_Parts:CRCW040250K0FKED -> Main_Board-rescue:CRCW040250K0FKED-SamacSys_Parts
Changed lines of the file:
@@
 $EndComp
 $Comp
-L SamacSys_Parts:CRCW040250K0FKED R9
+L Main_Board-rescue:CRCW040250K0FKED-SamacSys_Parts R9
 U 1 1 62263B47
 P 1000 9350
@@
 S2[2]
 $Comp
-L SamacSys_Parts:CRCW040250K0FKED R10
+L Main_Board-rescue:CRCW040250K0FKED-SamacSys_Parts R10
 U 1 1 62370C66
 P 1250 9350
@@
 $EndComp
 $Comp
-L SamacSys_Parts:CRCW040250K0FKED R11
+L Main_Board-rescue:CRCW040250K0FKED-SamacSys_Parts R11
 U 1 1 623712AF
 P 1500 9350
@@
 $EndComp
 $Comp
-L SamacSys_Parts:CRCW040250K0FKED R12
+L Main_Board-rescue:CRCW040250K0FKED-SamacSys_Parts R12
 U 1 1 623717A7
 P 1700 9350
@@
 $EndComp
 $Comp
-L SamacSys_Parts:CRCW040250K0FKED R13
+L Main_Board-rescue:CRCW040250K0FKED-SamacSys_Parts R13
 U 1 1 62371BCC
 P 1950 9350
@@
 $EndComp
 $Comp
-L SamacSys_Parts:CRCW040250K0FKED R14
+L Main_Board-rescue:CRCW040250K0FKED-SamacSys_Parts R14
 U 1 1 623720F0
 P 2150 9350
@@
 $EndComp
 $Comp
-L SamacSys_Parts:CRCW040250K0FKED R15
+L Main_Board-rescue:CRCW040250K0FKED-SamacSys_Parts R15
 U 1 1 6237253B
 P 2350 9350
@@
 $EndComp
 $Comp
-L SamacSys_Parts:CRCW040250K0FKED R16
+L Main_Board-rescue:CRCW040250K0FKED-SamacSys_Parts R16
 U 1 1 62372846
 P 2550 9350
@@
 $EndComp
 $Comp
-L SamacSys_Parts:CRCW040250K0FKED R17
+L Main_Board-rescue:CRCW040250K0FKED-SamacSys_Parts R17
 U 1 1 62372D0D
 P 2750 9350

Commit message: Updated Button
Connections:
- net GND: now also nRST1.1; no longer nRST1.3
- net nRST: now also nRST1.3; no longer nRST1.1
Other:
- moved on the sheet: nRST1
Changed lines of the file:
@@
 Wire Wire Line
 	1600 5650 1600 5750
-Wire Wire Line
-	1600 5750 2100 5750
 Connection ~ 1600 5750
 Wire Wire Line
 	1600 5750 1600 5850
 Wire Wire Line
-	1600 6550 1800 6550
-Wire Wire Line
 	1800 6550 1800 6600
-Wire Wire Line
-	2200 6550 2100 6550
 Connection ~ 1800 6550
 $Comp
@@
 $EndComp
 Wire Wire Line
-	2200 5750 2350 5750
-Wire Wire Line
 	2350 5750 2350 5700
-Connection ~ 2200 5750
 Text GLabel 2350 5700 1    50   Input ~ 0
 nRST
@@
 L Main_Board-rescue:PTS647SM50SMTR2LFS-SamacSys_Parts nRST1
 U 1 1 627772E3
-P 2200 5750
-F 0 "nRST1" V 2554 5878 50  0000 L CNN
-F 1 "A" V 2645 5878 50  0001 L CNN
-F 2 "PTS647SM50SMTR2LFS" H 2850 5850 50  0001 L CNN
-F 3 "https://www.ckswitches.com/media/2567/pts647.pdf" H 2850 5750 50  0001 L CNN
-F 4 "Tactile Switches 50mA 12VDC, 1.8N 5.0mm H, G leads" H 2850 5650 50  0001 L CNN "Description"
-F 5 "5.25" H 2850 5550 50  0001 L CNN "Height"
-F 6 "611-PTS647SM50SMTR2L" H 2850 5450 50  0001 L CNN "Mouser Part Number"
-F 7 "https://www.mouser.co.uk/ProductDetail/CK/PTS647SM50SMTR2LFS?qs=PqoDHHvF64%252BjK4ZB7f42kw%3D%3D" H 2850 5350 50  0001 L CNN "Mouser Price/Stock"
-F 8 "C & K COMPONENTS" H 2850 5250 50  0001 L CNN "Manufacturer_Name"
-F 9 "PTS647SM50SMTR2LFS" H 2850 5150 50  0001 L CNN "Manufacturer_Part_Number"
-	1    2200 5750
-	0    1    1    0
-$EndComp
-Wire Wire Line
-	2200 5750 2100 5750
-Connection ~ 2100 5750
-Connection ~ 2100 6550
-Wire Wire Line
-	2100 6550 1800 6550
+P 2550 6250
+F 0 "nRST1" V 2904 6378 50  0000 L CNN
+F 1 "A" V 2995 6378 50  0001 L CNN
+F 2 "PTS647SM50SMTR2LFS" H 3200 6350 50  0001 L CNN
+F 3 "https://www.ckswitches.com/media/2567/pts647.pdf" H 3200 6250 50  0001 L CNN
+F 4 "Tactile Switches 50mA 12VDC, 1.8N 5.0mm H, G leads" H 3200 6150 50  0001 L CNN "Description"
+F 5 "5.25" H 3200 6050 50  0001 L CNN "Height"
+F 6 "611-PTS647SM50SMTR2L" H 3200 5950 50  0001 L CNN "Mouser Part Number"
+F 7 "https://www.mouser.co.uk/ProductDetail/CK/PTS647SM50SMTR2LFS?qs=PqoDHHvF64%252BjK4ZB7f42kw%3D%3D" H 3200 5850 50  0001 L CNN "Mouser Price/Stock"
+F 8 "C & K COMPONENTS" H 3200 5750 50  0001 L CNN "Manufacturer_Name"
+F 9 "PTS647SM50SMTR2LFS" H 3200 5650 50  0001 L CNN "Manufacturer_Part_Number"
+	1    2550 6250
+	-1   0    0    1
+$EndComp
 Wire Wire Line
 	1600 6050 1600 6550
@@
 Wire Wire Line
 	6450 6150 6450 6200
+Wire Wire Line
+	1600 5750 2200 5750
+Wire Wire Line
+	2550 6150 2550 5800
+Wire Wire Line
+	2550 5800 2200 5800
+Wire Wire Line
+	2200 5800 2200 5750
+Connection ~ 2200 5750
+Wire Wire Line
+	2200 5750 2350 5750
+Wire Wire Line
+	2200 5800 1750 5800
+Wire Wire Line
+	1750 5800 1750 6150
+Connection ~ 2200 5800
+Wire Wire Line
+	1750 6250 1750 6550
+Wire Wire Line
+	1600 6550 1750 6550
+Connection ~ 1750 6550
+Wire Wire Line
+	1750 6550 1800 6550
+Wire Wire Line
+	2550 6250 2550 6550
+Wire Wire Line
+	1800 6550 2550 6550
 $EndSCHEMATC
