File: led_sensor/led_sensor.sch (KiCad schematic (older format))
At the start: 45 parts

Commit message: A
Parts:
- LED0, LED1, LED2, LED3, LED4, LED5, LED6, LED7: footprint LED Lib:XCXZCFBB53W-8VF -> SamacSys_Parts:HSMA-C380
Changed lines of the file:
@@
 F 0 "LED0" V 4096 4872 50  0000 R CNN
 F 1 "XZCFBB53W-8VF" V 4005 4872 50  0000 R CNN
-F 2 "LED Lib:XCXZCFBB53W-8VF" H 4050 5100 50  0001 C CNN
+F 2 "SamacSys_Parts:HSMA-C380" H 4050 5100 50  0001 C CNN
 F 3 "" H 4050 5100 50  0001 C CNN
 	1    4050 5100
@@
 F 0 "LED1" V 5196 4872 50  0000 R CNN
 F 1 "XZCFBB53W-8VF" V 5105 4872 50  0000 R CNN
-F 2 "LED Lib:XCXZCFBB53W-8VF" H 5150 5100 50  0001 C CNN
+F 2 "SamacSys_Parts:HSMA-C380" H 5150 5100 50  0001 C CNN
 F 3 "" H 5150 5100 50  0001 C CNN
 	1    5150 5100
@@
 F 0 "LED2" V 5704 5038 50  0000 L CNN
 F 1 "XZCFBB53W-8VF" V 5795 5038 50  0000 L CNN
-F 2 "LED Lib:XCXZCFBB53W-8VF" H 5750 5100 50  0001 C CNN
+F 2 "SamacSys_Parts:HSMA-C380" H 5750 5100 50  0001 C CNN
 F 3 "" H 5750 5100 50  0001 C CNN
 	1    5750 5100
@@
 F 0 "LED3" H 6800 5175 50  0000 C CNN
 F 1 "XZCFBB53W-8VF" V 6800 5084 50  0000 C CNN
-F 2 "LED Lib:XCXZCFBB53W-8VF" H 6800 5100 50  0001 C CNN
+F 2 "SamacSys_Parts:HSMA-C380" H 6800 5100 50  0001 C CNN
 F 3 "" H 6800 5100 50  0001 C CNN
 	1    6800 5100
@@
 F 0 "LED6" V 9404 5038 50  0000 L CNN
 F 1 "XZCFBB53W-8VF" V 9495 5038 50  0000 L CNN
-F 2 "LED Lib:XCXZCFBB53W-8VF" H 9450 5100 50  0001 C CNN
+F 2 "SamacSys_Parts:HSMA-C380" H 9450 5100 50  0001 C CNN
 F 3 "" H 9450 5100 50  0001 C CNN
 	1    9450 5100
@@
 F 0 "LED7" H 10350 5175 50  0000 C CNN
 F 1 "XZCFBB53W-8VF" H 10350 5084 50  0000 C CNN
-F 2 "LED Lib:XCXZCFBB53W-8VF" H 10350 5100 50  0001 C CNN
+F 2 "SamacSys_Parts:HSMA-C380" H 10350 5100 50  0001 C CNN
 F 3 "" H 10350 5100 50  0001 C CNN
 	1    10350 5100
@@
 F 0 "LED4" V 7896 4872 50  0000 R CNN
 F 1 "XZCFBB53W-8VF" V 7805 4872 50  0000 R CNN
-F 2 "LED Lib:XCXZCFBB53W-8VF" H 7850 5100 50  0001 C CNN
+F 2 "SamacSys_Parts:HSMA-C380" H 7850 5100 50  0001 C CNN
 F 3 "" H 7850 5100 50  0001 C CNN
 	1    7850 5100
@@
 F 0 "LED5" V 8646 4872 50  0000 R CNN
 F 1 "XZCFBB53W-8VF" V 8555 4872 50  0000 R CNN
-F 2 "LED Lib:XCXZCFBB53W-8VF" H 8600 5100 50  0001 C CNN
+F 2 "SamacSys_Parts:HSMA-C380" H 8600 5100 50  0001 C CNN
 F 3 "" H 8600 5100 50  0001 C CNN
 	1    8600 5100

Commit message: more library changes
Parts:
- H#0, H#7, U#1, U#2, U#3, U#4, U#5, U#6: symbol HallSensor:AH3362Q -> led_sensor-rescue:AH3362Q-HallSensor
- HM#1: symbol SN74HCS151QPWRQ1:SN74HCS151QPWRQ1 -> led_sensor-rescue:SN74HCS151QPWRQ1-SN74HCS151QPWRQ1
- LED0, LED1, LED2, LED3, LED4, LED5, LED6, LED7: symbol xzcfbb53w-8vf:XZCFBB53W-8VF -> led_sensor-rescue:XZCFBB53W-8VF-xzcfbb53w-8vf
Changed lines of the file:
@@
 $EndDescr
 $Comp
-L SN74HCS151QPWRQ1:SN74HCS151QPWRQ1 HM#1
+L led_sensor-rescue:SN74HCS151QPWRQ1-SN74HCS151QPWRQ1 HM#1
 U 1 1 615917A2
 P 3300 2950
@@
 	2600 3950 2600 4400
 $Comp
-L HallSensor:AH3362Q H#0
+L led_sensor-rescue:AH3362Q-HallSensor H#0
 U 1 1 615A38AC
 P 4750 3350
@@
 $EndComp
 $Comp
-L HallSensor:AH3362Q U#1
+L led_sensor-rescue:AH3362Q-HallSensor U#1
 U 1 1 615A5ADB
 P 5500 3350
@@
 $EndComp
 $Comp
-L HallSensor:AH3362Q U#2
+L led_sensor-rescue:AH3362Q-HallSensor U#2
 U 1 1 615A5DEF
 P 6150 3350
@@
 $EndComp
 $Comp
-L HallSensor:AH3362Q U#3
+L led_sensor-rescue:AH3362Q-HallSensor U#3
 U 1 1 615A6394
 P 6800 3350
@@
 $EndComp
 $Comp
-L HallSensor:AH3362Q U#4
+L led_sensor-rescue:AH3362Q-HallSensor U#4
 U 1 1 615A67A4
 P 7500 3350
@@
 $EndComp
 $Comp
-L HallSensor:AH3362Q U#5
+L led_sensor-rescue:AH3362Q-HallSensor U#5
 U 1 1 615A6E92
 P 8200 3350
@@
 $EndComp
 $Comp
-L HallSensor:AH3362Q U#6
+L led_sensor-rescue:AH3362Q-HallSensor U#6
 U 1 1 615A72E7
 P 8850 3350
@@
 	8600 4100 8600 3700
 $Comp
-L HallSensor:AH3362Q H#7
+L led_sensor-rescue:AH3362Q-HallSensor H#7
 U 1 1 615B3333
 P 9500 3350
@@
 	9250 4150 9250 3700
 $Comp
-L xzcfbb53w-8vf:XZCFBB53W-8VF LED0
+L led_sensor-rescue:XZCFBB53W-8VF-xzcfbb53w-8vf LED0
 U 1 1 6153BA49
 P 4050 5100
@@
 $EndComp
 $Comp
-L xzcfbb53w-8vf:XZCFBB53W-8VF LED1
+L led_sensor-rescue:XZCFBB53W-8VF-xzcfbb53w-8vf LED1
 U 1 1 6153D881
 P 5150 5100
@@
 $EndComp
 $Comp
-L xzcfbb53w-8vf:XZCFBB53W-8VF LED2
+L led_sensor-rescue:XZCFBB53W-8VF-xzcfbb53w-8vf LED2
 U 1 1 6153E4EA
 P 5750 5100
@@
 $EndComp
 $Comp
-L xzcfbb53w-8vf:XZCFBB53W-8VF LED3
+L led_sensor-rescue:XZCFBB53W-8VF-xzcfbb53w-8vf LED3
 U 1 1 615401E5
 P 6800 5100
@@
 $EndComp
 $Comp
-L xzcfbb53w-8vf:XZCFBB53W-8VF LED6
+L led_sensor-rescue:XZCFBB53W-8VF-xzcfbb53w-8vf LED6
 U 1 1 61544A04
 P 9450 5100
@@
 $EndComp
 $Comp
-L xzcfbb53w-8vf:XZCFBB53W-8VF LED7
+L led_sensor-rescue:XZCFBB53W-8VF-xzcfbb53w-8vf LED7
 U 1 1 61544A0A
 P 10350 5100
@@
 din
 $Comp
-L xzcfbb53w-8vf:XZCFBB53W-8VF LED4
+L led_sensor-rescue:XZCFBB53W-8VF-xzcfbb53w-8vf LED4
 U 1 1 615449F8
 P 7850 5100
@@
 Connection ~ 8450 5350
 $Comp
-L xzcfbb53w-8vf:XZCFBB53W-8VF LED5
+L led_sensor-rescue:XZCFBB53W-8VF-xzcfbb53w-8vf LED5
 U 1 1 615449FE
 P 8600 5100

Commit message: 8 Hall Sensor
Parts:
- H#0, H#7, U#1, U#2, U#3, U#4, U#5, U#6: symbol led_sensor-rescue:AH3362Q-HallSensor -> HallSensor:AH3362Q
- HM#1: symbol led_sensor-rescue:SN74HCS151QPWRQ1-SN74HCS151QPWRQ1 -> SN74HCS151QPWRQ1:SN74HCS151QPWRQ1
- LED0, LED1, LED2, LED3, LED4, LED5, LED6, LED7: symbol led_sensor-rescue:XZCFBB53W-8VF-xzcfbb53w-8vf -> xzcfbb53w-8vf:XZCFBB53W-8VF
Changed lines of the file:
@@
 $EndDescr
 $Comp
-L led_sensor-rescue:SN74HCS151QPWRQ1-SN74HCS151QPWRQ1 HM#1
+L SN74HCS151QPWRQ1:SN74HCS151QPWRQ1 HM#1
 U 1 1 615917A2
 P 3300 2950
@@
 	2600 3950 2600 4400
 $Comp
-L led_sensor-rescue:AH3362Q-HallSensor H#0
+L HallSensor:AH3362Q H#0
 U 1 1 615A38AC
 P 4750 3350
@@
 $EndComp
 $Comp
-L led_sensor-rescue:AH3362Q-HallSensor U#1
+L HallSensor:AH3362Q U#1
 U 1 1 615A5ADB
 P 5500 3350
@@
 $EndComp
 $Comp
-L led_sensor-rescue:AH3362Q-HallSensor U#2
+L HallSensor:AH3362Q U#2
 U 1 1 615A5DEF
 P 6150 3350
@@
 $EndComp
 $Comp
-L led_sensor-rescue:AH3362Q-HallSensor U#3
+L HallSensor:AH3362Q U#3
 U 1 1 615A6394
 P 6800 3350
@@
 $EndComp
 $Comp
-L led_sensor-rescue:AH3362Q-HallSensor U#4
+L HallSensor:AH3362Q U#4
 U 1 1 615A67A4
 P 7500 3350
@@
 $EndComp
 $Comp
-L led_sensor-rescue:AH3362Q-HallSensor U#5
+L HallSensor:AH3362Q U#5
 U 1 1 615A6E92
 P 8200 3350
@@
 $EndComp
 $Comp
-L led_sensor-rescue:AH3362Q-HallSensor U#6
+L HallSensor:AH3362Q U#6
 U 1 1 615A72E7
 P 8850 3350
@@
 	8600 4100 8600 3700
 $Comp
-L led_sensor-rescue:AH3362Q-HallSensor H#7
+L HallSensor:AH3362Q H#7
 U 1 1 615B3333
 P 9500 3350
@@
 	9250 4150 9250 3700
 $Comp
-L led_sensor-rescue:XZCFBB53W-8VF-xzcfbb53w-8vf LED0
+L xzcfbb53w-8vf:XZCFBB53W-8VF LED0
 U 1 1 6153BA49
 P 4050 5100
@@
 $EndComp
 $Comp
-L led_sensor-rescue:XZCFBB53W-8VF-xzcfbb53w-8vf LED1
+L xzcfbb53w-8vf:XZCFBB53W-8VF LED1
 U 1 1 6153D881
 P 5150 5100
@@
 $EndComp
 $Comp
-L led_sensor-rescue:XZCFBB53W-8VF-xzcfbb53w-8vf LED2
+L xzcfbb53w-8vf:XZCFBB53W-8VF LED2
 U 1 1 6153E4EA
 P 5750 5100
@@
 $EndComp
 $Comp
-L led_sensor-rescue:XZCFBB53W-8VF-xzcfbb53w-8vf LED3
+L xzcfbb53w-8vf:XZCFBB53W-8VF LED3
 U 1 1 615401E5
 P 6800 5100
@@
 $EndComp
 $Comp
-L led_sensor-rescue:XZCFBB53W-8VF-xzcfbb53w-8vf LED6
+L xzcfbb53w-8vf:XZCFBB53W-8VF LED6
 U 1 1 61544A04
 P 9450 5100
@@
 $EndComp
 $Comp
-L led_sensor-rescue:XZCFBB53W-8VF-xzcfbb53w-8vf LED7
+L xzcfbb53w-8vf:XZCFBB53W-8VF LED7
 U 1 1 61544A0A
 P 10350 5100
@@
 din
 $Comp
-L led_sensor-rescue:XZCFBB53W-8VF-xzcfbb53w-8vf LED4
+L xzcfbb53w-8vf:XZCFBB53W-8VF LED4
 U 1 1 615449F8
 P 7850 5100
@@
 Connection ~ 8450 5350
 $Comp
-L led_sensor-rescue:XZCFBB53W-8VF-xzcfbb53w-8vf LED5
+L xzcfbb53w-8vf:XZCFBB53W-8VF LED5
 U 1 1 615449FE
 P 8600 5100

Commit message: fixed reverse biased LEDs
Parts:
- H#0, H#7, U#1, U#2, U#3, U#4, U#5, U#6: symbol HallSensor:AH3362Q -> led_sensor-rescue:AH3362Q-HallSensor
- HM#1: symbol SN74HCS151QPWRQ1:SN74HCS151QPWRQ1 -> led_sensor-rescue:SN74HCS151QPWRQ1-SN74HCS151QPWRQ1
- LED0, LED1, LED2, LED3, LED4, LED5, LED6, LED7: symbol xzcfbb53w-8vf:XZCFBB53W-8VF -> led_sensor-rescue:XZCFBB53W-8VF-xzcfbb53w-8vf
Connections:
- net CCin: now also LED0.1 (-), LED1.1 (-), LED2.1 (-), LED3.1 (-), LED4.1 (-), LED5.1 (-), LED6.1 (-), LED7.1 (-); no longer LED0.2 (+), LED1.2 (+), LED2.2 (+), LED3.2 (+), LED4.2 (+), LED5.2 (+), LED6.2 (+), LED7.2 (+)
- net ain: now also LED7.2 (+); no longer LED7.1 (-)
- net bin: now also LED6.2 (+); no longer LED6.1 (-)
- net cin: now also LED5.2 (+); no longer LED5.1 (-)
- net din: now also LED4.2 (+); no longer LED4.1 (-)
- net dpin: now also LED0.2 (+); no longer LED0.1 (-)
- net ein: now also LED3.2 (+); no longer LED3.1 (-)
- net fin: now also LED2.2 (+); no longer LED2.1 (-)
- net gin: now also LED1.2 (+); no longer LED1.1 (-)
Changed lines of the file:
@@
 $EndDescr
 $Comp
-L SN74HCS151QPWRQ1:SN74HCS151QPWRQ1 HM#1
+L led_sensor-rescue:SN74HCS151QPWRQ1-SN74HCS151QPWRQ1 HM#1
 U 1 1 615917A2
 P 3300 2950
@@
 	2600 3950 2600 4400
 $Comp
-L HallSensor:AH3362Q H#0
+L led_sensor-rescue:AH3362Q-HallSensor H#0
 U 1 1 615A38AC
 P 4750 3350
@@
 $EndComp
 $Comp
-L HallSensor:AH3362Q U#1
+L led_sensor-rescue:AH3362Q-HallSensor U#1
 U 1 1 615A5ADB
 P 5500 3350
@@
 $EndComp
 $Comp
-L HallSensor:AH3362Q U#2
+L led_sensor-rescue:AH3362Q-HallSensor U#2
 U 1 1 615A5DEF
 P 6150 3350
@@
 $EndComp
 $Comp
-L HallSensor:AH3362Q U#3
+L led_sensor-rescue:AH3362Q-HallSensor U#3
 U 1 1 615A6394
 P 6800 3350
@@
 $EndComp
 $Comp
-L HallSensor:AH3362Q U#4
+L led_sensor-rescue:AH3362Q-HallSensor U#4
 U 1 1 615A67A4
 P 7500 3350
@@
 $EndComp
 $Comp
-L HallSensor:AH3362Q U#5
+L led_sensor-rescue:AH3362Q-HallSensor U#5
 U 1 1 615A6E92
 P 8200 3350
@@
 $EndComp
 $Comp
-L HallSensor:AH3362Q U#6
+L led_sensor-rescue:AH3362Q-HallSensor U#6
 U 1 1 615A72E7
 P 8850 3350
@@
 	8600 4100 8600 3700
 $Comp
-L HallSensor:AH3362Q H#7
+L led_sensor-rescue:AH3362Q-HallSensor H#7
 U 1 1 615B3333
 P 9500 3350
@@
 	9250 4150 9250 3700
 $Comp
-L xzcfbb53w-8vf:XZCFBB53W-8VF LED0
+L led_sensor-rescue:XZCFBB53W-8VF-xzcfbb53w-8vf LED0
 U 1 1 6153BA49
-P 4050 5100
-F 0 "LED0" V 4096 4872 50  0000 R CNN
-F 1 "XZCFBB53W-8VF" V 4005 4872 50  0000 R CNN
-F 2 "SamacSys_Parts:HSMA-C380" H 4050 5100 50  0001 C CNN
-F 3 "" H 4050 5100 50  0001 C CNN
-	1    4050 5100
-	0    1    1    0
-$EndComp
-$Comp
-L xzcfbb53w-8vf:XZCFBB53W-8VF LED1
+P 3750 5100
+F 0 "LED0" H 3750 5050 50  0000 R CNN
+F 1 "XZCFBB53W-8VF" H 3700 4850 50  0000 R CNN
+F 2 "SamacSys_Parts:HSMA-C380" H 3750 5100 50  0001 C CNN
+F 3 "" H 3750 5100 50  0001 C CNN
+	1    3750 5100
+	0    -1   -1   0
+$EndComp
+$Comp
+L led_sensor-rescue:XZCFBB53W-8VF-xzcfbb53w-8vf LED1
 U 1 1 6153D881
-P 5150 5100
-F 0 "LED1" V 5196 4872 50  0000 R CNN
-F 1 "XZCFBB53W-8VF" V 5105 4872 50  0000 R CNN
-F 2 "SamacSys_Parts:HSMA-C380" H 5150 5100 50  0001 C CNN
-F 3 "" H 5150 5100 50  0001 C CNN
-	1    5150 5100
-	0    1    1    0
-$EndComp
-$Comp
-L xzcfbb53w-8vf:XZCFBB53W-8VF LED2
+P 4850 5100
+F 0 "LED1" H 4900 5150 50  0000 R CNN
+F 1 "XZCFBB53W-8VF" H 5100 5050 50  0000 R CNN
+F 2 "SamacSys_Parts:HSMA-C380" H 4850 5100 50  0001 C CNN
+F 3 "" H 4850 5100 50  0001 C CNN
+	1    4850 5100
+	0    -1   -1   0
+$EndComp
+$Comp
+L led_sensor-rescue:XZCFBB53W-8VF-xzcfbb53w-8vf LED2
 U 1 1 6153E4EA
-P 5750 5100
-F 0 "LED2" V 5704 5038 50  0000 L CNN
-F 1 "XZCFBB53W-8VF" V 5795 5038 50  0000 L CNN
-F 2 "SamacSys_Parts:HSMA-C380" H 5750 5100 50  0001 C CNN
-F 3 "" H 5750 5100 50  0001 C CNN
-	1    5750 5100
-	0    1    1    0
-$EndComp
-$Comp
-L xzcfbb53w-8vf:XZCFBB53W-8VF LED3
+P 5450 5100
+F 0 "LED2" H 5404 5038 50  0000 L CNN
+F 1 "XZCFBB53W-8VF" H 5050 4850 50  0000 L CNN
+F 2 "SamacSys_Parts:HSMA-C380" H 5450 5100 50  0001 C CNN
+F 3 "" H 5450 5100 50  0001 C CNN
+	1    5450 5100
+	0    -1   -1   0
+$EndComp
+$Comp
+L led_sensor-rescue:XZCFBB53W-8VF-xzcfbb53w-8vf LED3
 U 1 1 615401E5
-P 6800 5100
-F 0 "LED3" H 6800 5175 50  0000 C CNN
-F 1 "XZCFBB53W-8VF" V 6800 5084 50  0000 C CNN
-F 2 "SamacSys_Parts:HSMA-C380" H 6800 5100 50  0001 C CNN
-F 3 "" H 6800 5100 50  0001 C CNN
-	1    6800 5100
-	0    1    1    0
-$EndComp
-$Comp
-L xzcfbb53w-8vf:XZCFBB53W-8VF LED6
+P 6500 5100
+F 0 "LED3" H 6500 5175 50  0000 C CNN
+F 1 "XZCFBB53W-8VF" H 6500 5050 50  0000 C CNN
+F 2 "SamacSys_Parts:HSMA-C380" H 6500 5100 50  0001 C CNN
+F 3 "" H 6500 5100 50  0001 C CNN
+	1    6500 5100
+	0    -1   -1   0
+$EndComp
+$Comp
+L led_sensor-rescue:XZCFBB53W-8VF-xzcfbb53w-8vf LED6
 U 1 1 61544A04
-P 9450 5100
-F 0 "LED6" V 9404 5038 50  0000 L CNN
-F 1 "XZCFBB53W-8VF" V 9495 5038 50  0000 L CNN
-F 2 "SamacSys_Parts:HSMA-C380" H 9450 5100 50  0001 C CNN
-F 3 "" H 9450 5100 50  0001 C CNN
-	1    9450 5100
-	0    1    1    0
-$EndComp
-$Comp
-L xzcfbb53w-8vf:XZCFBB53W-8VF LED7
+P 9150 5100
+F 0 "LED6" H 9104 5038 50  0000 L CNN
+F 1 "XZCFBB53W-8VF" H 8800 5100 50  0000 L CNN
+F 2 "SamacSys_Parts:HSMA-C380" H 9150 5100 50  0001 C CNN
+F 3 "" H 9150 5100 50  0001 C CNN
+	1    9150 5100
+	0    -1   -1   0
+$EndComp
+$Comp
+L led_sensor-rescue:XZCFBB53W-8VF-xzcfbb53w-8vf LED7
 U 1 1 61544A0A
-P 10350 5100
-F 0 "LED7" H 10350 5175 50  0000 C CNN
-F 1 "XZCFBB53W-8VF" H 10350 5084 50  0000 C CNN
-F 2 "SamacSys_Parts:HSMA-C380" H 10350 5100 50  0001 C CNN
-F 3 "" H 10350 5100 50  0001 C CNN
-	1    10350 5100
-	0    1    1    0
+P 10050 5100
+F 0 "LED7" H 10050 5175 50  0000 C CNN
+F 1 "XZCFBB53W-8VF" H 10050 5084 50  0000 C CNN
+F 2 "SamacSys_Parts:HSMA-C380" H 10050 5100 50  0001 C CNN
+F 3 "" H 10050 5100 50  0001 C CNN
+	1    10050 5100
+	0    -1   -1   0
 $EndComp
 Text Label 5000 4550 1    50   ~ 0
@@
 din
 $Comp
-L xzcfbb53w-8vf:XZCFBB53W-8VF LED4
+L led_sensor-rescue:XZCFBB53W-8VF-xzcfbb53w-8vf LED4
 U 1 1 615449F8
-P 7850 5100
-F 0 "LED4" V 7896 4872 50  0000 R CNN
-F 1 "XZCFBB53W-8VF" V 7805 4872 50  0000 R CNN
-F 2 "SamacSys_Parts:HSMA-C380" H 7850 5100 50  0001 C CNN
-F 3 "" H 7850 5100 50  0001 C CNN
-	1    7850 5100
-	0    1    1    0
+P 7550 5100
+F 0 "LED4" H 7600 5100 50  0000 R CNN
+F 1 "XZCFBB53W-8VF" H 7700 4850 50  0000 R CNN
+F 2 "SamacSys_Parts:HSMA-C380" H 7550 5100 50  0001 C CNN
+F 3 "" H 7550 5100 50  0001 C CNN
+	1    7550 5100
+	0    -1   -1   0
 $EndComp
 Wire Wire Line
@@
 Connection ~ 7150 5350
 Connection ~ 7700 5350
-Connection ~ 9300 5350
-Wire Wire Line
-	9300 5350 10200 5350
 Text Label 7150 4350 0    50   ~ 0
 CCin
@@
 Connection ~ 3900 4550
 Wire Wire Line
-	8450 5350 9300 5350
-Wire Wire Line
 	7700 5350 8450 5350
 Connection ~ 8450 5350
 $Comp
-L xzcfbb53w-8vf:XZCFBB53W-8VF LED5
+L led_sensor-rescue:XZCFBB53W-8VF-xzcfbb53w-8vf LED5
 U 1 1 615449FE
-P 8600 5100
-F 0 "LED5" V 8646 4872 50  0000 R CNN
-F 1 "XZCFBB53W-8VF" V 8555 4872 50  0000 R CNN
-F 2 "SamacSys_Parts:HSMA-C380" H 8600 5100 50  0001 C CNN
-F 3 "" H 8600 5100 50  0001 C CNN
-	1    8600 5100
-	0    1    1    0
+P 8300 5100
+F 0 "LED5" H 8346 4872 50  0000 R CNN
+F 1 "XZCFBB53W-8VF" H 8550 5050 50  0000 R CNN
+F 2 "SamacSys_Parts:HSMA-C380" H 8300 5100 50  0001 C CNN
+F 3 "" H 8300 5100 50  0001 C CNN
+	1    8300 5100
+	0    -1   -1   0
 $EndComp
 $Comp
@@
 	10200 4700 10250 4700
 Connection ~ 10250 4600
+Wire Wire Line
+	8450 5350 9300 5350
+Connection ~ 9300 5350
+Wire Wire Line
+	9300 5350 10200 5350
 $EndSCHEMATC

Commit message: screenshots
Other:
- note added: "Circuit"
- note added: "Mounting Equipment"
Changed lines of the file:
@@
 Wire Wire Line
 	9300 5350 10200 5350
+Text Notes 1650 700  0    50   ~ 0
+Mounting Equipment
+Wire Notes Line
+	700  1450 700  550
+Wire Notes Line
+	700  550  2500 550
+Wire Notes Line
+	2500 550  2500 1450
+Wire Notes Line
+	2500 1450 700  1450
+Wire Notes Line
+	700  1500 10750 1500
+Wire Notes Line
+	10750 1500 10750 5900
+Wire Notes Line
+	10750 5900 700  5900
+Wire Notes Line
+	700  1500 700  6000
+Text Notes 8900 2150 0    197  ~ 0
+Circuit
 $EndSCHEMATC
