File: led_sensor/led_sensor.sch (KiCad schematic (older format))
At the start: 54 parts

Commit message: switched symbols
Parts:
- LED1, LED2, LED3, LED4, LED5, LED6, LED7: symbol led_sensor-rescue:XZCFBB53W-8VF-xzcfbb53w-8vf -> xzcfbb53w-8vf:XZCFBB53W-8VF
- U1: renamed from LED0; value XZCFBB53W-8VF -> XZCFBB53W-8VF-xzcfbb53w-8vf; symbol led_sensor-rescue:XZCFBB53W-8VF-xzcfbb53w-8vf -> xzcfbb53w-8vf:XZCFBB53W-8VF
Changed lines of the file:
@@
 	2900 4150 9250 4150
 $Comp
-L led_sensor-rescue:XZCFBB53W-8VF-xzcfbb53w-8vf LED0
+L xzcfbb53w-8vf:XZCFBB53W-8VF U1
 U 1 1 6153BA49
 P 3750 5100
-F 0 "LED0" H 3750 5050 50  0000 R CNN
-F 1 "XZCFBB53W-8VF" H 3700 4850 50  0000 R CNN
+F 0 "U1" H 3750 5050 50  0000 R CNN
+F 1 "XZCFBB53W-8VF-xzcfbb53w-8vf" H 3700 4850 50  0000 R CNN
 F 2 "SamacSys_Parts:HSMA-C380" H 3750 5100 50  0001 C CNN
 F 3 "" H 3750 5100 50  0001 C CNN
@@
 $EndComp
 $Comp
-L led_sensor-rescue:XZCFBB53W-8VF-xzcfbb53w-8vf LED1
+L xzcfbb53w-8vf:XZCFBB53W-8VF LED1
 U 1 1 6153D881
 P 4850 5100
@@
 $EndComp
 $Comp
-L led_sensor-rescue:XZCFBB53W-8VF-xzcfbb53w-8vf LED2
+L xzcfbb53w-8vf:XZCFBB53W-8VF LED2
 U 1 1 6153E4EA
 P 5450 5100
@@
 $EndComp
 $Comp
-L led_sensor-rescue:XZCFBB53W-8VF-xzcfbb53w-8vf LED3
+L xzcfbb53w-8vf:XZCFBB53W-8VF LED3
 U 1 1 615401E5
 P 6500 5100
@@
 $EndComp
 $Comp
-L led_sensor-rescue:XZCFBB53W-8VF-xzcfbb53w-8vf LED6
+L xzcfbb53w-8vf:XZCFBB53W-8VF LED6
 U 1 1 61544A04
 P 9150 5100
@@
 $EndComp
 $Comp
-L led_sensor-rescue:XZCFBB53W-8VF-xzcfbb53w-8vf LED7
+L xzcfbb53w-8vf:XZCFBB53W-8VF LED7
 U 1 1 61544A0A
 P 10050 5100
@@
 din
 $Comp
-L led_sensor-rescue:XZCFBB53W-8VF-xzcfbb53w-8vf LED4
+L xzcfbb53w-8vf:XZCFBB53W-8VF LED4
 U 1 1 615449F8
 P 7550 5100
@@
 Connection ~ 8450 5350
 $Comp
-L led_sensor-rescue:XZCFBB53W-8VF-xzcfbb53w-8vf LED5
+L xzcfbb53w-8vf:XZCFBB53W-8VF LED5
 U 1 1 615449FE
 P 8300 5100

Commit message: final Rev1 changes. increased heatsink area, flipped LEDs again, increased button mount hole size
Parts:
- LED1, LED2, LED3, LED4, LED5, LED6, LED7, U1: symbol xzcfbb53w-8vf:XZCFBB53W-8VF -> led_sensor-rescue:XZCFBB53W-8VF-xzcfbb53w-8vf
Connections:
- net CCin: now also LED1.2 (-), LED2.2 (-), LED3.2 (-), LED4.2 (-), LED5.2 (-), LED6.2 (-), LED7.2 (-), U1.2 (-); no longer LED1.1 (+), LED2.1 (+), LED3.1 (+), LED4.1 (+), LED5.1 (+), LED6.1 (+), LED7.1 (+), U1.1 (+)
- net ain: now also LED7.1 (+); no longer LED7.2 (-)
- net bin: now also LED6.1 (+); no longer LED6.2 (-)
- net cin: now also LED5.1 (+); no longer LED5.2 (-)
- net din: now also LED4.1 (+); no longer LED4.2 (-)
- net dpin: now also U1.1 (+); no longer U1.2 (-)
- net ein: now also LED3.1 (+); no longer LED3.2 (-)
- net fin: now also LED2.1 (+); no longer LED2.2 (-)
- net gin: now also LED1.1 (+); no longer LED1.2 (-)
Changed lines of the file:
@@
 	2900 4150 9250 4150
 $Comp
-L xzcfbb53w-8vf:XZCFBB53W-8VF U1
+L led_sensor-rescue:XZCFBB53W-8VF-xzcfbb53w-8vf U1
 U 1 1 6153BA49
-P 3750 5100
-F 0 "U1" H 3750 5050 50  0000 R CNN
-F 1 "XZCFBB53W-8VF-xzcfbb53w-8vf" H 3700 4850 50  0000 R CNN
-F 2 "SamacSys_Parts:HSMA-C380" H 3750 5100 50  0001 C CNN
-F 3 "" H 3750 5100 50  0001 C CNN
-	1    3750 5100
-	0    -1   -1   0
-$EndComp
-$Comp
-L xzcfbb53w-8vf:XZCFBB53W-8VF LED1
-U 1 1 6153D881
-P 4850 5100
-F 0 "LED1" H 4900 5150 50  0000 R CNN
-F 1 "XZCFBB53W-8VF" H 5100 5050 50  0000 R CNN
-F 2 "SamacSys_Parts:HSMA-C380" H 4850 5100 50  0001 C CNN
-F 3 "" H 4850 5100 50  0001 C CNN
-	1    4850 5100
-	0    -1   -1   0
-$EndComp
-$Comp
-L xzcfbb53w-8vf:XZCFBB53W-8VF LED2
+P 4050 5100
+F 0 "U1" H 4050 5050 50  0000 R CNN
+F 1 "XZCFBB53W-8VF-xzcfbb53w-8vf" H 4950 4850 50  0000 R CNN
+F 2 "SamacSys_Parts:HSMA-C380" H 4050 5100 50  0001 C CNN
+F 3 "" H 4050 5100 50  0001 C CNN
+	1    4050 5100
+	0    1    1    0
+$EndComp
+$Comp
+L led_sensor-rescue:XZCFBB53W-8VF-xzcfbb53w-8vf LED2
 U 1 1 6153E4EA
-P 5450 5100
-F 0 "LED2" H 5404 5038 50  0000 L CNN
-F 1 "XZCFBB53W-8VF" H 5050 4850 50  0000 L CNN
-F 2 "SamacSys_Parts:HSMA-C380" H 5450 5100 50  0001 C CNN
-F 3 "" H 5450 5100 50  0001 C CNN
-	1    5450 5100
-	0    -1   -1   0
-$EndComp
-$Comp
-L xzcfbb53w-8vf:XZCFBB53W-8VF LED3
+P 5750 5100
+F 0 "LED2" H 5704 5038 50  0000 L CNN
+F 1 "XZCFBB53W-8VF" H 5350 4850 50  0000 L CNN
+F 2 "SamacSys_Parts:HSMA-C380" H 5750 5100 50  0001 C CNN
+F 3 "" H 5750 5100 50  0001 C CNN
+	1    5750 5100
+	0    1    1    0
+$EndComp
+$Comp
+L led_sensor-rescue:XZCFBB53W-8VF-xzcfbb53w-8vf LED3
 U 1 1 615401E5
-P 6500 5100
-F 0 "LED3" H 6500 5175 50  0000 C CNN
-F 1 "XZCFBB53W-8VF" H 6500 5050 50  0000 C CNN
-F 2 "SamacSys_Parts:HSMA-C380" H 6500 5100 50  0001 C CNN
-F 3 "" H 6500 5100 50  0001 C CNN
-	1    6500 5100
-	0    -1   -1   0
-$EndComp
-$Comp
-L xzcfbb53w-8vf:XZCFBB53W-8VF LED6
+P 6800 5100
+F 0 "LED3" H 6800 5175 50  0000 C CNN
+F 1 "XZCFBB53W-8VF" H 6800 5050 50  0000 C CNN
+F 2 "SamacSys_Parts:HSMA-C380" H 6800 5100 50  0001 C CNN
+F 3 "" H 6800 5100 50  0001 C CNN
+	1    6800 5100
+	0    1    1    0
+$EndComp
+$Comp
+L led_sensor-rescue:XZCFBB53W-8VF-xzcfbb53w-8vf LED6
 U 1 1 61544A04
-P 9150 5100
-F 0 "LED6" H 9104 5038 50  0000 L CNN
-F 1 "XZCFBB53W-8VF" H 8800 5100 50  0000 L CNN
-F 2 "SamacSys_Parts:HSMA-C380" H 9150 5100 50  0001 C CNN
-F 3 "" H 9150 5100 50  0001 C CNN
-	1    9150 5100
-	0    -1   -1   0
-$EndComp
-$Comp
-L xzcfbb53w-8vf:XZCFBB53W-8VF LED7
+P 9450 5100
+F 0 "LED6" H 9404 5038 50  0000 L CNN
+F 1 "XZCFBB53W-8VF" H 9100 5100 50  0000 L CNN
+F 2 "SamacSys_Parts:HSMA-C380" H 9450 5100 50  0001 C CNN
+F 3 "" H 9450 5100 50  0001 C CNN
+	1    9450 5100
+	0    1    1    0
+$EndComp
+$Comp
+L led_sensor-rescue:XZCFBB53W-8VF-xzcfbb53w-8vf LED7
 U 1 1 61544A0A
-P 10050 5100
-F 0 "LED7" H 10050 5175 50  0000 C CNN
-F 1 "XZCFBB53W-8VF" H 10050 5084 50  0000 C CNN
-F 2 "SamacSys_Parts:HSMA-C380" H 10050 5100 50  0001 C CNN
-F 3 "" H 10050 5100 50  0001 C CNN
-	1    10050 5100
-	0    -1   -1   0
+P 10350 5100
+F 0 "LED7" H 10350 5175 50  0000 C CNN
+F 1 "XZCFBB53W-8VF" H 10350 5084 50  0000 C CNN
+F 2 "SamacSys_Parts:HSMA-C380" H 10350 5100 50  0001 C CNN
+F 3 "" H 10350 5100 50  0001 C CNN
+	1    10350 5100
+	0    1    1    0
 $EndComp
 Text Label 5000 4550 1    50   ~ 0
@@
 din
 $Comp
-L xzcfbb53w-8vf:XZCFBB53W-8VF LED4
+L led_sensor-rescue:XZCFBB53W-8VF-xzcfbb53w-8vf LED4
 U 1 1 615449F8
-P 7550 5100
-F 0 "LED4" H 7600 5100 50  0000 R CNN
-F 1 "XZCFBB53W-8VF" H 7700 4850 50  0000 R CNN
-F 2 "SamacSys_Parts:HSMA-C380" H 7550 5100 50  0001 C CNN
-F 3 "" H 7550 5100 50  0001 C CNN
-	1    7550 5100
-	0    -1   -1   0
+P 7850 5100
+F 0 "LED4" H 7900 5100 50  0000 R CNN
+F 1 "XZCFBB53W-8VF" H 8000 4850 50  0000 R CNN
+F 2 "SamacSys_Parts:HSMA-C380" H 7850 5100 50  0001 C CNN
+F 3 "" H 7850 5100 50  0001 C CNN
+	1    7850 5100
+	0    1    1    0
 $EndComp
 Wire Wire Line
 	7150 5350 6650 5350
-Connection ~ 5000 5350
-Wire Wire Line
-	5000 5350 3900 5350
 Connection ~ 5600 5350
-Wire Wire Line
-	5600 5350 5000 5350
 Connection ~ 6650 5350
 Wire Wire Line
@@
 Connection ~ 8450 5350
 $Comp
-L xzcfbb53w-8vf:XZCFBB53W-8VF LED5
+L led_sensor-rescue:XZCFBB53W-8VF-xzcfbb53w-8vf LED5
 U 1 1 615449FE
-P 8300 5100
-F 0 "LED5" H 8346 4872 50  0000 R CNN
-F 1 "XZCFBB53W-8VF" H 8550 5050 50  0000 R CNN
-F 2 "SamacSys_Parts:HSMA-C380" H 8300 5100 50  0001 C CNN
-F 3 "" H 8300 5100 50  0001 C CNN
-	1    8300 5100
-	0    -1   -1   0
+P 8600 5100
+F 0 "LED5" H 8646 4872 50  0000 R CNN
+F 1 "XZCFBB53W-8VF" H 8850 5050 50  0000 R CNN
+F 2 "SamacSys_Parts:HSMA-C380" H 8600 5100 50  0001 C CNN
+F 3 "" H 8600 5100 50  0001 C CNN
+	1    8600 5100
+	0    1    1    0
 $EndComp
 $Comp
@@
 	5150 3150 5800 3150
 Wire Wire Line
-	3300 4350 3300 4600
+	3300 4350 3300 4550
 Connection ~ 3300 4350
 $Comp
@@
 Wire Wire Line
 	6200 4250 6350 4250
+Wire Wire Line
+	5600 5350 5000 5350
+Wire Wire Line
+	5000 5350 3900 5350
+Connection ~ 5000 5350
+$Comp
+L led_sensor-rescue:XZCFBB53W-8VF-xzcfbb53w-8vf LED1
+U 1 1 6153D881
+P 5150 5100
+F 0 "LED1" H 5200 5150 50  0000 R CNN
+F 1 "XZCFBB53W-8VF" H 5400 5050 50  0000 R CNN
+F 2 "SamacSys_Parts:HSMA-C380" H 5150 5100 50  0001 C CNN
+F 3 "" H 5150 5100 50  0001 C CNN
+	1    5150 5100
+	0    1    1    0
+$EndComp
+$Comp
+L power:PWR_FLAG #FLG0101
+U 1 1 61694F37
+P 3300 4550
+F 0 "#FLG0101" H 3300 4625 50  0001 C CNN
+F 1 "PWR_FLAG" V 3300 4677 50  0000 L CNN
+F 2 "" H 3300 4550 50  0001 C CNN
+F 3 "~" H 3300 4550 50  0001 C CNN
+	1    3300 4550
+	0    -1   -1   0
+$EndComp
+Connection ~ 3300 4550
+Wire Wire Line
+	3300 4550 3300 4600
 $EndSCHEMATC
